File: Generated_Project/Rev3_8Seat_PCBWay_Chassis_v1/MI250X_8OAM_PCBWay_Chassis_Stub.kicad_pcb (KiCad board)
At the start: 4 copper layers, 492 x 372 mm, 48 parts, among them J0_Conn0 218910-1115, J0_Conn1 218910-1115, J1_Conn0 218910-1115, J1_Conn1 218910-1115, J2_Conn0 218910-1115, J2_Conn1 218910-1115, J3_Conn0 218910-1115, J3_Conn1 218910-1115, J4_Conn0 218910-1115, J4_Conn1 218910-1115, J5_Conn0 218910-1115, J5_Conn1 218910-1115, J6_Conn0 218910-1115, J6_Conn1 218910-1115, J7_Conn0 218910-1115, J7_Conn1 218910-1115

Commit message: Raise Rev3 chassis to 8 electrically designed seats.
Name v1.0 power/PE/clock nets on all eight OAM seats toward two DNP
PM8536B-FEI (x8 per GCD), keep SB175 star + local P48V pours, and generate
the 12-layer 2.0 mm stuffed-switch target. First stuffing may still populate
two modules; the PCB does not need a respin for the other six.

Do not fabricate. Do not energize P48V.

Co-authored-by: zivzancoeli-commits <zivzancoeli-commits@users.noreply.github.com>
Parts:
- added J_SB175: SB175_175A_600V, footprints:Anderson_SB175_2pole, F.Cu at (70.0, 362.0)
Connections:
- J0_Conn0 pad A11: OAM0_S1_RX10P -> (no net)
- J0_Conn0 pad A12: OAM0_S1_RX10N -> (no net)
- J0_Conn0 pad A15: OAM0_S1_RX8P -> (no net)
- J0_Conn0 pad A16: OAM0_S1_RX8N -> (no net)
- J0_Conn0 pad A19: OAM0_S2_RX13P -> (no net)
- J0_Conn0 pad A20: OAM0_S2_RX13N -> (no net)
- J0_Conn0 pad A23: OAM0_S2_RX11P -> (no net)
- J0_Conn0 pad A24: OAM0_S2_RX11N -> (no net)
- J0_Conn0 pad A27: OAM0_S2_RX9P -> (no net)
- J0_Conn0 pad A28: OAM0_S2_RX9N -> (no net)
- J0_Conn0 pad A31: OAM0_S3_RX14P -> (no net)
- J0_Conn0 pad A32: OAM0_S3_RX14N -> (no net)
- J0_Conn0 pad A35: OAM0_S3_RX11P -> (no net)
- J0_Conn0 pad A36: OAM0_S3_RX11N -> (no net)
- J0_Conn0 pad A39: OAM0_S3_RX9P -> (no net)
- J0_Conn0 pad A40: OAM0_S3_RX9N -> (no net)
- J0_Conn0 pad A7: OAM0_S1_RX13P -> (no net)
- J0_Conn0 pad A8: OAM0_S1_RX13N -> (no net)
- J0_Conn0 pad B10: OAM0_S1_RX12N -> (no net)
- J0_Conn0 pad B13: OAM0_S1_RX9P -> (no net)
- J0_Conn0 pad B14: OAM0_S1_RX9N -> (no net)
- J0_Conn0 pad B17: OAM0_S2_RX15P -> (no net)
- J0_Conn0 pad B18: OAM0_S2_RX15N -> (no net)
- J0_Conn0 pad B21: OAM0_S2_RX12P -> (no net)
- J0_Conn0 pad B22: OAM0_S2_RX12N -> (no net)
- J0_Conn0 pad B25: OAM0_S2_RX10P -> (no net)
- J0_Conn0 pad B26: OAM0_S2_RX10N -> (no net)
- J0_Conn0 pad B29: OAM0_S2_RX8P -> (no net)
- J0_Conn0 pad B30: OAM0_S2_RX8N -> (no net)
- J0_Conn0 pad B33: OAM0_S3_RX13P -> (no net)
- J0_Conn0 pad B34: OAM0_S3_RX13N -> (no net)
- J0_Conn0 pad B37: OAM0_S3_RX10P -> (no net)
- J0_Conn0 pad B38: OAM0_S3_RX10N -> (no net)
- J0_Conn0 pad B41: OAM0_S3_RX8P -> (no net)
- J0_Conn0 pad B42: OAM0_S3_RX8N -> (no net)
- J0_Conn0 pad B5: OAM0_S1_RX15P -> (no net)
- J0_Conn0 pad B6: OAM0_S1_RX15N -> (no net)
- J0_Conn0 pad B9: OAM0_S1_RX12P -> (no net)
- J0_Conn0 pad C11: OAM0_S1_RX11P -> (no net)
- J0_Conn0 pad C12: OAM0_S1_RX11N -> (no net)
- J0_Conn0 pad C15: OAM0_S1_RX1P -> (no net)
- J0_Conn0 pad C16: OAM0_S1_RX1N -> (no net)
- J0_Conn0 pad C19: OAM0_S2_RX14P -> (no net)
- J0_Conn0 pad C20: OAM0_S2_RX14N -> (no net)
- J0_Conn0 pad C23: OAM0_S2_RX4P -> (no net)
- J0_Conn0 pad C24: OAM0_S2_RX4N -> (no net)
- J0_Conn0 pad C27: OAM0_S2_RX1P -> (no net)
- J0_Conn0 pad C28: OAM0_S2_RX1N -> (no net)
- J0_Conn0 pad C31: OAM0_S3_RX15P -> (no net)
- J0_Conn0 pad C32: OAM0_S3_RX15N -> (no net)
- J0_Conn0 pad C35: OAM0_S3_RX12P -> (no net)
- J0_Conn0 pad C36: OAM0_S3_RX12N -> (no net)
- J0_Conn0 pad C39: OAM0_S3_RX2P -> (no net)
- J0_Conn0 pad C40: OAM0_S3_RX2N -> (no net)
- J0_Conn0 pad C7: OAM0_S1_RX14P -> (no net)
- J0_Conn0 pad C8: OAM0_S1_RX14N -> (no net)
- J0_Conn0 pad D10: OAM0_S1_RX5N -> (no net)
- J0_Conn0 pad D13: OAM0_S1_RX3P -> (no net)
- J0_Conn0 pad D14: OAM0_S1_RX3N -> (no net)
- J0_Conn0 pad D17: OAM0_S1_RX0P -> (no net)
- J0_Conn0 pad D18: OAM0_S1_RX0N -> (no net)
- J0_Conn0 pad D21: OAM0_S2_RX6P -> (no net)
- J0_Conn0 pad D22: OAM0_S2_RX6N -> (no net)
- J0_Conn0 pad D25: OAM0_S2_RX3P -> (no net)
- J0_Conn0 pad D26: OAM0_S2_RX3N -> (no net)
- J0_Conn0 pad D29: OAM0_S2_RX0P -> (no net)
- J0_Conn0 pad D30: OAM0_S2_RX0N -> (no net)
- J0_Conn0 pad D33: OAM0_S3_RX6P -> (no net)
- J0_Conn0 pad D34: OAM0_S3_RX6N -> (no net)
- J0_Conn0 pad D37: OAM0_S3_RX4P -> (no net)
- J0_Conn0 pad D38: OAM0_S3_RX4N -> (no net)
- J0_Conn0 pad D41: OAM0_S3_RX1P -> (no net)
- J0_Conn0 pad D42: OAM0_S3_RX1N -> (no net)
- J0_Conn0 pad D5: OAM0_S1_RX7P -> (no net)
- J0_Conn0 pad D6: OAM0_S1_RX7N -> (no net)
- J0_Conn0 pad D9: OAM0_S1_RX5P -> (no net)
- J0_Conn0 pad E11: OAM0_S1_RX4P -> (no net)
- J0_Conn0 pad E12: OAM0_S1_RX4N -> (no net)
- J0_Conn0 pad E15: OAM0_S1_RX2P -> (no net)
- J0_Conn0 pad E16: OAM0_S1_RX2N -> (no net)
- J0_Conn0 pad E19: OAM0_S2_RX7P -> (no net)
- J0_Conn0 pad E20: OAM0_S2_RX7N -> (no net)
- J0_Conn0 pad E23: OAM0_S2_RX5P -> (no net)
- J0_Conn0 pad E24: OAM0_S2_RX5N -> (no net)
- J0_Conn0 pad E27: OAM0_S2_RX2P -> (no net)
- J0_Conn0 pad E28: OAM0_S2_RX2N -> (no net)
- J0_Conn0 pad E31: OAM0_S3_RX7P -> (no net)
- J0_Conn0 pad E32: OAM0_S3_RX7N -> (no net)
- J0_Conn0 pad E35: OAM0_S3_RX5P -> (no net)
- J0_Conn0 pad E36: OAM0_S3_RX5N -> (no net)
- J0_Conn0 pad E39: OAM0_S3_RX3P -> (no net)
- J0_Conn0 pad E40: OAM0_S3_RX3N -> (no net)
- J0_Conn0 pad E43: OAM0_S3_RX0P -> (no net)
- J0_Conn0 pad E44: OAM0_S3_RX0N -> (no net)
- J0_Conn0 pad E7: OAM0_S1_RX6P -> (no net)
- J0_Conn0 pad E8: OAM0_S1_RX6N -> (no net)
- J0_Conn0 pad G11: OAM0_S1_TX10P -> (no net)
- J0_Conn0 pad G12: OAM0_S1_TX10N -> (no net)
- J0_Conn0 pad G15: OAM0_S1_TX8P -> (no net)
- J0_Conn0 pad G16: OAM0_S1_TX8N -> (no net)
- J0_Conn0 pad G19: OAM0_S2_TX13P -> (no net)
- J0_Conn0 pad G20: OAM0_S2_TX13N -> (no net)
- J0_Conn0 pad G23: OAM0_S2_TX11P -> (no net)
- J0_Conn0 pad G24: OAM0_S2_TX11N -> (no net)
- J0_Conn0 pad G27: OAM0_S2_TX9P -> (no net)
- J0_Conn0 pad G28: OAM0_S2_TX9N -> (no net)
- J0_Conn0 pad G31: OAM0_S3_TX14P -> (no net)
- J0_Conn0 pad G32: OAM0_S3_TX14N -> (no net)
- J0_Conn0 pad G35: OAM0_S3_TX12P -> (no net)
- J0_Conn0 pad G36: OAM0_S3_TX12N -> (no net)
- J0_Conn0 pad G39: OAM0_S3_TX10P -> (no net)
- J0_Conn0 pad G40: OAM0_S3_TX10N -> (no net)
- J0_Conn0 pad G43: OAM0_S3_TX8P -> (no net)
- J0_Conn0 pad G44: OAM0_S3_TX8N -> (no net)
- J0_Conn0 pad G7: OAM0_S1_TX13P -> (no net)
- J0_Conn0 pad G8: OAM0_S1_TX13N -> (no net)
- J0_Conn0 pad H10: OAM0_S1_TX12N -> (no net)
- J0_Conn0 pad H13: OAM0_S1_TX9P -> (no net)
- J0_Conn0 pad H14: OAM0_S1_TX9N -> (no net)
- J0_Conn0 pad H17: OAM0_S2_TX15P -> (no net)
- J0_Conn0 pad H18: OAM0_S2_TX15N -> (no net)
- J0_Conn0 pad H21: OAM0_S2_TX12P -> (no net)
- J0_Conn0 pad H22: OAM0_S2_TX12N -> (no net)
- J0_Conn0 pad H25: OAM0_S2_TX10P -> (no net)
- J0_Conn0 pad H26: OAM0_S2_TX10N -> (no net)
- J0_Conn0 pad H29: OAM0_S2_TX8P -> (no net)
- J0_Conn0 pad H30: OAM0_S2_TX8N -> (no net)
- J0_Conn0 pad H33: OAM0_S3_TX13P -> (no net)
- J0_Conn0 pad H34: OAM0_S3_TX13N -> (no net)
- J0_Conn0 pad H37: OAM0_S3_TX11P -> (no net)
- J0_Conn0 pad H38: OAM0_S3_TX11N -> (no net)
- J0_Conn0 pad H41: OAM0_S3_TX9P -> (no net)
- J0_Conn0 pad H42: OAM0_S3_TX9N -> (no net)
- J0_Conn0 pad H5: OAM0_S1_TX15P -> (no net)
- J0_Conn0 pad H6: OAM0_S1_TX15N -> (no net)
- J0_Conn0 pad H9: OAM0_S1_TX12P -> (no net)
- J0_Conn0 pad J11: OAM0_S1_TX11P -> (no net)
- J0_Conn0 pad J12: OAM0_S1_TX11N -> (no net)
- J0_Conn0 pad J15: OAM0_S1_TX1P -> (no net)
- J0_Conn0 pad J16: OAM0_S1_TX1N -> (no net)
- J0_Conn0 pad J19: OAM0_S2_TX14P -> (no net)
- J0_Conn0 pad J20: OAM0_S2_TX14N -> (no net)
- J0_Conn0 pad J23: OAM0_S2_TX4P -> (no net)
- J0_Conn0 pad J24: OAM0_S2_TX4N -> (no net)
- J0_Conn0 pad J27: OAM0_S2_TX1P -> (no net)
- J0_Conn0 pad J28: OAM0_S2_TX1N -> (no net)
- J0_Conn0 pad J31: OAM0_S3_TX15P -> (no net)
- J0_Conn0 pad J32: OAM0_S3_TX15N -> (no net)
- J0_Conn0 pad J35: OAM0_S3_TX4P -> (no net)
- J0_Conn0 pad J36: OAM0_S3_TX4N -> (no net)
- J0_Conn0 pad J39: OAM0_S3_TX1P -> (no net)
- J0_Conn0 pad J40: OAM0_S3_TX1N -> (no net)
- J0_Conn0 pad J7: OAM0_S1_TX14P -> (no net)
- J0_Conn0 pad J8: OAM0_S1_TX14N -> (no net)
- J0_Conn0 pad K10: OAM0_S1_TX5N -> (no net)
- J0_Conn0 pad K13: OAM0_S1_TX3P -> (no net)
- J0_Conn0 pad K14: OAM0_S1_TX3N -> (no net)
- J0_Conn0 pad K17: OAM0_S1_TX0P -> (no net)
- J0_Conn0 pad K18: OAM0_S1_TX0N -> (no net)
- J0_Conn0 pad K21: OAM0_S2_TX6P -> (no net)
- J0_Conn0 pad K22: OAM0_S2_TX6N -> (no net)
- J0_Conn0 pad K25: OAM0_S2_TX3P -> (no net)
- J0_Conn0 pad K26: OAM0_S2_TX3N -> (no net)
- J0_Conn0 pad K29: OAM0_S2_TX0P -> (no net)
- J0_Conn0 pad K30: OAM0_S2_TX0N -> (no net)
- J0_Conn0 pad K33: OAM0_S3_TX6P -> (no net)
- J0_Conn0 pad K34: OAM0_S3_TX6N -> (no net)
- J0_Conn0 pad K37: OAM0_S3_TX3P -> (no net)
- J0_Conn0 pad K38: OAM0_S3_TX3N -> (no net)
- J0_Conn0 pad K41: OAM0_S3_TX0P -> (no net)
- J0_Conn0 pad K42: OAM0_S3_TX0N -> (no net)
- J0_Conn0 pad K5: OAM0_S1_TX7P -> (no net)
- J0_Conn0 pad K6: OAM0_S1_TX7N -> (no net)
- J0_Conn0 pad K9: OAM0_S1_TX5P -> (no net)
- J0_Conn0 pad L11: OAM0_S1_TX4P -> (no net)
- J0_Conn0 pad L12: OAM0_S1_TX4N -> (no net)
- J0_Conn0 pad L15: OAM0_S1_TX2P -> (no net)
- J0_Conn0 pad L16: OAM0_S1_TX2N -> (no net)
- J0_Conn0 pad L19: OAM0_S2_TX7P -> (no net)
- J0_Conn0 pad L20: OAM0_S2_TX7N -> (no net)
- J0_Conn0 pad L23: OAM0_S2_TX5P -> (no net)
- J0_Conn0 pad L24: OAM0_S2_TX5N -> (no net)
- J0_Conn0 pad L27: OAM0_S2_TX2P -> (no net)
- J0_Conn0 pad L28: OAM0_S2_TX2N -> (no net)
- J0_Conn0 pad L31: OAM0_S3_TX7P -> (no net)
- J0_Conn0 pad L32: OAM0_S3_TX7N -> (no net)
- J0_Conn0 pad L35: OAM0_S3_TX5P -> (no net)
- J0_Conn0 pad L36: OAM0_S3_TX5N -> (no net)
- J0_Conn0 pad L39: OAM0_S3_TX2P -> (no net)
- J0_Conn0 pad L40: OAM0_S3_TX2N -> (no net)
- J0_Conn0 pad L7: OAM0_S1_TX6P -> (no net)
- J0_Conn0 pad L8: OAM0_S1_TX6N -> (no net)
- J0_Conn1 pad A11: OAM0_S7_TX5N -> (no net)
- J0_Conn1 pad A12: OAM0_S7_TX5P -> (no net)
- J0_Conn1 pad A15: OAM0_S7_TX2N -> (no net)
- J0_Conn1 pad A16: OAM0_S7_TX2P -> (no net)
- J0_Conn1 pad A19: OAM0_S7_TX0N -> (no net)
- J0_Conn1 pad A20: OAM0_S7_TX0P -> (no net)
- J0_Conn1 pad A23: OAM0_S6_TX3N -> (no net)
- J0_Conn1 pad A24: OAM0_S6_TX3P -> (no net)
- J0_Conn1 pad A27: OAM0_S6_TX5N -> (no net)
- J0_Conn1 pad A28: OAM0_S6_TX5P -> (no net)
- J0_Conn1 pad A3: OAM0_CONN1_INITMODE -> (no net)
- J0_Conn1 pad A31: OAM0_S6_TX7N -> (no net)
- J0_Conn1 pad A32: OAM0_S6_TX7P -> (no net)
- J0_Conn1 pad A35: OAM0_S5_TX2N -> (no net)
- J0_Conn1 pad A36: OAM0_S5_TX2P -> (no net)
- J0_Conn1 pad A39: OAM0_S5_TX4N -> (no net)
- J0_Conn1 pad A4: OAM0_CONN1_INT# -> (no net)
- J0_Conn1 pad A40: OAM0_S5_TX4P -> (no net)
- J0_Conn1 pad A43: OAM0_S5_TX6N -> (no net)
- J0_Conn1 pad A44: OAM0_S5_TX6P -> (no net)
- J0_Conn1 pad A47: OAM0_S4_TX1N -> (no net)
- J0_Conn1 pad A48: OAM0_S4_TX1P -> (no net)
- J0_Conn1 pad A51: OAM0_S4_TX3N -> (no net)
- J0_Conn1 pad A52: OAM0_S4_TX3P -> (no net)
- J0_Conn1 pad A55: OAM0_S4_TX5N -> (no net)
- J0_Conn1 pad A56: OAM0_S4_TX5P -> (no net)
- J0_Conn1 pad A59: OAM0_S4_TX7N -> (no net)
- J0_Conn1 pad A60: OAM0_S4_TX7P -> (no net)
- J0_Conn1 pad B10: OAM0_S7_TX7P -> (no net)
- J0_Conn1 pad B13: OAM0_S7_TX4N -> (no net)
- J0_Conn1 pad B14: OAM0_S7_TX4P -> (no net)
- J0_Conn1 pad B17: OAM0_S7_TX1N -> (no net)
- J0_Conn1 pad B18: OAM0_S7_TX1P -> (no net)
- J0_Conn1 pad B21: OAM0_S6_TX1N -> (no net)
- J0_Conn1 pad B22: OAM0_S6_TX1P -> (no net)
- J0_Conn1 pad B25: OAM0_S6_TX4N -> (no net)
- J0_Conn1 pad B26: OAM0_S6_TX4P -> (no net)
- J0_Conn1 pad B29: OAM0_S6_TX6N -> (no net)
- J0_Conn1 pad B30: OAM0_S6_TX6P -> (no net)
- J0_Conn1 pad B33: OAM0_S5_TX0N -> (no net)
- J0_Conn1 pad B34: OAM0_S5_TX0P -> (no net)
- J0_Conn1 pad B37: OAM0_S5_TX3N -> (no net)
- J0_Conn1 pad B38: OAM0_S5_TX3P -> (no net)
- J0_Conn1 pad B41: OAM0_S5_TX5N -> (no net)
- J0_Conn1 pad B42: OAM0_S5_TX5P -> (no net)
- J0_Conn1 pad B45: OAM0_S5_TX7N -> (no net)
- J0_Conn1 pad B46: OAM0_S5_TX7P -> (no net)
- J0_Conn1 pad B49: OAM0_S4_TX2N -> (no net)
- J0_Conn1 pad B50: OAM0_S4_TX2P -> (no net)
- J0_Conn1 pad B53: OAM0_S4_TX4N -> (no net)
- J0_Conn1 pad B54: OAM0_S4_TX4P -> (no net)
- J0_Conn1 pad B57: OAM0_S4_TX6N -> (no net)
- J0_Conn1 pad B58: OAM0_S4_TX6P -> (no net)
- J0_Conn1 pad B9: OAM0_S7_TX7N -> (no net)
- J0_Conn1 pad C11: OAM0_S7_TX6N -> (no net)
- J0_Conn1 pad C12: OAM0_S7_TX6P -> (no net)
- J0_Conn1 pad C15: OAM0_S7_TX3N -> (no net)
- J0_Conn1 pad C16: OAM0_S7_TX3P -> (no net)
- J0_Conn1 pad C19: OAM0_S6_TX0N -> (no net)
- J0_Conn1 pad C20: OAM0_S6_TX0P -> (no net)
- J0_Conn1 pad C23: OAM0_S6_TX2N -> (no net)
- J0_Conn1 pad C24: OAM0_S6_TX2P -> (no net)
- J0_Conn1 pad C27: OAM0_S6_TX13N -> (no net)
- J0_Conn1 pad C28: OAM0_S6_TX13P -> (no net)
- J0_Conn1 pad C31: OAM0_S6_TX15N -> (no net)
- J0_Conn1 pad C32: OAM0_S6_TX15P -> (no net)
- J0_Conn1 pad C35: OAM0_S5_TX1N -> (no net)
- J0_Conn1 pad C36: OAM0_S5_TX1P -> (no net)
- J0_Conn1 pad C39: OAM0_S5_TX11N -> (no net)
- J0_Conn1 pad C40: OAM0_S5_TX11P -> (no net)
- J0_Conn1 pad C43: OAM0_S5_TX14N -> (no net)
- J0_Conn1 pad C44: OAM0_S5_TX14P -> (no net)
- J0_Conn1 pad C47: OAM0_S4_TX0N -> (no net)
- J0_Conn1 pad C48: OAM0_S4_TX0P -> (no net)
- J0_Conn1 pad C51: OAM0_S4_TX11N -> (no net)
- J0_Conn1 pad C52: OAM0_S4_TX11P -> (no net)
- J0_Conn1 pad C55: OAM0_S4_TX14N -> (no net)
- J0_Conn1 pad C56: OAM0_S4_TX14P -> (no net)
- J0_Conn1 pad D1: OAM0_CONN1_MODPRS# -> (no net)
- J0_Conn1 pad D10: OAM0_S7_TX12P -> (no net)
- J0_Conn1 pad D13: OAM0_S7_TX10N -> (no net)
- J0_Conn1 pad D14: OAM0_S7_TX10P -> (no net)
- J0_Conn1 pad D17: OAM0_S7_TX8N -> (no net)
- J0_Conn1 pad D18: OAM0_S7_TX8P -> (no net)
- J0_Conn1 pad D2: OAM0_CONN1_MODSEL# -> (no net)
- J0_Conn1 pad D21: OAM0_S6_TX9N -> (no net)
- J0_Conn1 pad D22: OAM0_S6_TX9P -> (no net)
- J0_Conn1 pad D25: OAM0_S6_TX11N -> (no net)
- J0_Conn1 pad D26: OAM0_S6_TX11P -> (no net)
- J0_Conn1 pad D29: OAM0_S6_TX14N -> (no net)
- J0_Conn1 pad D30: OAM0_S6_TX14P -> (no net)
- J0_Conn1 pad D33: OAM0_S5_TX8N -> (no net)
- J0_Conn1 pad D34: OAM0_S5_TX8P -> (no net)
- J0_Conn1 pad D37: OAM0_S5_TX10N -> (no net)
- J0_Conn1 pad D38: OAM0_S5_TX10P -> (no net)
- J0_Conn1 pad D41: OAM0_S5_TX12N -> (no net)
- J0_Conn1 pad D42: OAM0_S5_TX12P -> (no net)
- J0_Conn1 pad D45: OAM0_S5_TX15N -> (no net)
- J0_Conn1 pad D46: OAM0_S5_TX15P -> (no net)
- J0_Conn1 pad D49: OAM0_S4_TX9N -> (no net)
- J0_Conn1 pad D5: OAM0_S7_TX14N -> (no net)
- J0_Conn1 pad D50: OAM0_S4_TX9P -> (no net)
- J0_Conn1 pad D53: OAM0_S4_TX12N -> (no net)
- J0_Conn1 pad D54: OAM0_S4_TX12P -> (no net)
- J0_Conn1 pad D57: OAM0_S4_TX15N -> (no net)
- J0_Conn1 pad D58: OAM0_S4_TX15P -> (no net)
- J0_Conn1 pad D6: OAM0_S7_TX14P -> (no net)
- J0_Conn1 pad D61: OAM0_MNGMT_LINK0TN -> (no net)
- J0_Conn1 pad D62: OAM0_MNGMT_LINK0TP -> (no net)
- J0_Conn1 pad D9: OAM0_S7_TX12N -> (no net)
- J0_Conn1 pad E11: OAM0_S7_TX11N -> (no net)
- J0_Conn1 pad E12: OAM0_S7_TX11P -> (no net)
- J0_Conn1 pad E15: OAM0_S7_TX9N -> (no net)
- J0_Conn1 pad E16: OAM0_S7_TX9P -> (no net)
- J0_Conn1 pad E19: OAM0_S6_TX8N -> (no net)
- J0_Conn1 pad E20: OAM0_S6_TX8P -> (no net)
- J0_Conn1 pad E23: OAM0_S6_TX10N -> (no net)
- J0_Conn1 pad E24: OAM0_S6_TX10P -> (no net)
- J0_Conn1 pad E27: OAM0_S6_TX12N -> (no net)
- J0_Conn1 pad E28: OAM0_S6_TX12P -> (no net)
- J0_Conn1 pad E3: OAM0_S7_TX15N -> (no net)
- J0_Conn1 pad E35: OAM0_S5_TX9N -> (no net)
- J0_Conn1 pad E36: OAM0_S5_TX9P -> (no net)
- J0_Conn1 pad E4: OAM0_S7_TX15P -> (no net)
- J0_Conn1 pad E43: OAM0_S5_TX13N -> (no net)
- J0_Conn1 pad E44: OAM0_S5_TX13P -> (no net)
- J0_Conn1 pad E47: OAM0_S4_TX8N -> (no net)
- J0_Conn1 pad E48: OAM0_S4_TX8P -> (no net)
- J0_Conn1 pad E51: OAM0_S4_TX10N -> (no net)
- J0_Conn1 pad E52: OAM0_S4_TX10P -> (no net)
- J0_Conn1 pad E55: OAM0_S4_TX13N -> (no net)
- J0_Conn1 pad E56: OAM0_S4_TX13P -> (no net)
- J0_Conn1 pad E63: OAM0_MNGMT_LINK1TP -> (no net)
- J0_Conn1 pad E64: OAM0_MNGMT_LINK1TN -> (no net)
- J0_Conn1 pad E7: OAM0_S7_TX13N -> (no net)
- J0_Conn1 pad E8: OAM0_S7_TX13P -> (no net)
- J0_Conn1 pad F1: OAM0_CONN1_RESET# -> (no net)
- J0_Conn1 pad F10: OAM0_CONN2_YELLOW_LED -> (no net)
- J0_Conn1 pad F2: OAM0_CONN1_GREEN_LED -> (no net)
- J0_Conn1 pad F5: OAM0_CONN2_MODSEL# -> (no net)
- J0_Conn1 pad F6: OAM0_CONN2_RESET# -> (no net)
- J0_Conn1 pad F9: OAM0_CONN2_GREEN_LED -> (no net)
- J0_Conn1 pad G11: OAM0_S7_RX5N -> (no net)
- J0_Conn1 pad G12: OAM0_S7_RX5P -> (no net)
- J0_Conn1 pad G15: OAM0_S7_RX2N -> (no net)
- J0_Conn1 pad G16: OAM0_S7_RX2P -> (no net)
- J0_Conn1 pad G19: OAM0_S7_RX0N -> (no net)
- J0_Conn1 pad G20: OAM0_S7_RX0P -> (no net)
- J0_Conn1 pad G23: OAM0_S6_RX3N -> (no net)
- J0_Conn1 pad G24: OAM0_S6_RX3P -> (no net)
- J0_Conn1 pad G27: OAM0_S6_RX6N -> (no net)
- J0_Conn1 pad G28: OAM0_S6_RX6P -> (no net)
- J0_Conn1 pad G35: OAM0_S5_RX2N -> (no net)
- J0_Conn1 pad G36: OAM0_S5_RX2P -> (no net)
- J0_Conn1 pad G39: OAM0_S5_RX5N -> (no net)
- J0_Conn1 pad G40: OAM0_S5_RX5P -> (no net)
- J0_Conn1 pad G43: OAM0_S5_RX7N -> (no net)
- J0_Conn1 pad G44: OAM0_S5_RX7P -> (no net)
- J0_Conn1 pad G47: OAM0_S4_RX0N -> (no net)
- J0_Conn1 pad G48: OAM0_S4_RX0P -> (no net)
- J0_Conn1 pad G51: OAM0_S4_RX2N -> (no net)
- J0_Conn1 pad G52: OAM0_S4_RX2P -> (no net)
- J0_Conn1 pad G59: OAM0_S4_RX7N -> (no net)
- J0_Conn1 pad G60: OAM0_S4_RX7P -> (no net)
- J0_Conn1 pad G63: OAM0_MNGMT_LINK1RP -> (no net)
- J0_Conn1 pad G64: OAM0_MNGMT_LINK1RN -> (no net)
- J0_Conn1 pad H1: OAM0_CONN1_YELLOW_LED -> (no net)
- J0_Conn1 pad H10: OAM0_S7_RX7P -> (no net)
- J0_Conn1 pad H13: OAM0_S7_RX4N -> (no net)
- J0_Conn1 pad H14: OAM0_S7_RX4P -> (no net)
- J0_Conn1 pad H17: OAM0_S7_RX1N -> (no net)
- J0_Conn1 pad H18: OAM0_S7_RX1P -> (no net)
- J0_Conn1 pad H2: OAM0_CONN2_INITMODE -> (no net)
- J0_Conn1 pad H21: OAM0_S6_RX1N -> (no net)
- J0_Conn1 pad H22: OAM0_S6_RX1P -> (no net)
- J0_Conn1 pad H25: OAM0_S6_RX4N -> (no net)
- J0_Conn1 pad H26: OAM0_S6_RX4P -> (no net)
- J0_Conn1 pad H29: OAM0_S6_RX7N -> (no net)
- J0_Conn1 pad H30: OAM0_S6_RX7P -> (no net)
- J0_Conn1 pad H33: OAM0_S5_RX0N -> (no net)
- J0_Conn1 pad H34: OAM0_S5_RX0P -> (no net)
- J0_Conn1 pad H37: OAM0_S5_RX3N -> (no net)
- J0_Conn1 pad H38: OAM0_S5_RX3P -> (no net)
- J0_Conn1 pad H41: OAM0_S5_RX6N -> (no net)
- J0_Conn1 pad H42: OAM0_S5_RX6P -> (no net)
- J0_Conn1 pad H49: OAM0_S4_RX1N -> (no net)
- J0_Conn1 pad H50: OAM0_S4_RX1P -> (no net)
- J0_Conn1 pad H53: OAM0_S4_RX3N -> (no net)
- J0_Conn1 pad H54: OAM0_S4_RX3P -> (no net)
- J0_Conn1 pad H57: OAM0_S4_RX5N -> (no net)
- J0_Conn1 pad H58: OAM0_S4_RX5P -> (no net)
- J0_Conn1 pad H61: OAM0_MNGMT_LINK0RN -> (no net)
- J0_Conn1 pad H62: OAM0_MNGMT_LINK0RP -> (no net)
- J0_Conn1 pad H9: OAM0_S7_RX7N -> (no net)
- J0_Conn1 pad J11: OAM0_S7_RX6N -> (no net)
- J0_Conn1 pad J12: OAM0_S7_RX6P -> (no net)
- J0_Conn1 pad J15: OAM0_S7_RX3N -> (no net)
- J0_Conn1 pad J16: OAM0_S7_RX3P -> (no net)
- J0_Conn1 pad J19: OAM0_S6_RX0N -> (no net)
- J0_Conn1 pad J20: OAM0_S6_RX0P -> (no net)
- J0_Conn1 pad J23: OAM0_S6_RX2N -> (no net)
- J0_Conn1 pad J24: OAM0_S6_RX2P -> (no net)
- J0_Conn1 pad J27: OAM0_S6_RX5N -> (no net)
- J0_Conn1 pad J28: OAM0_S6_RX5P -> (no net)
- J0_Conn1 pad J31: OAM0_S6_RX15N -> (no net)
- J0_Conn1 pad J32: OAM0_S6_RX15P -> (no net)
- J0_Conn1 pad J35: OAM0_S5_RX1N -> (no net)
- J0_Conn1 pad J36: OAM0_S5_RX1P -> (no net)
- J0_Conn1 pad J39: OAM0_S5_RX4N -> (no net)
- J0_Conn1 pad J40: OAM0_S5_RX4P -> (no net)
- J0_Conn1 pad J43: OAM0_S5_RX14N -> (no net)
- J0_Conn1 pad J44: OAM0_S5_RX14P -> (no net)
- J0_Conn1 pad J47: OAM0_S4_RX9N -> (no net)
- J0_Conn1 pad J48: OAM0_S4_RX9P -> (no net)
- J0_Conn1 pad J51: OAM0_S4_RX12N -> (no net)
- J0_Conn1 pad J52: OAM0_S4_RX12P -> (no net)
- J0_Conn1 pad J55: OAM0_S4_RX4N -> (no net)
- J0_Conn1 pad J56: OAM0_S4_RX4P -> (no net)
- J0_Conn1 pad J59: OAM0_S4_RX6N -> (no net)
- J0_Conn1 pad J60: OAM0_S4_RX6P -> (no net)
- J0_Conn1 pad J7: OAM0_S7_RX13N -> (no net)
- J0_Conn1 pad J8: OAM0_S7_RX13P -> (no net)
- J0_Conn1 pad K10: OAM0_S7_RX12P -> (no net)
- J0_Conn1 pad K13: OAM0_S7_RX10N -> (no net)
- J0_Conn1 pad K14: OAM0_S7_RX10P -> (no net)
- J0_Conn1 pad K17: OAM0_S7_RX8N -> (no net)
- J0_Conn1 pad K18: OAM0_S7_RX8P -> (no net)
- J0_Conn1 pad K21: OAM0_S6_RX9N -> (no net)
- J0_Conn1 pad K22: OAM0_S6_RX9P -> (no net)
- J0_Conn1 pad K25: OAM0_S6_RX11N -> (no net)
- J0_Conn1 pad K26: OAM0_S6_RX11P -> (no net)
- J0_Conn1 pad K29: OAM0_S6_RX13N -> (no net)
- J0_Conn1 pad K30: OAM0_S6_RX13P -> (no net)
- J0_Conn1 pad K33: OAM0_S5_RX8N -> (no net)
- J0_Conn1 pad K34: OAM0_S5_RX8P -> (no net)
- J0_Conn1 pad K37: OAM0_S5_RX10N -> (no net)
- J0_Conn1 pad K38: OAM0_S5_RX10P -> (no net)
- J0_Conn1 pad K41: OAM0_S5_RX12N -> (no net)
- J0_Conn1 pad K42: OAM0_S5_RX12P -> (no net)
- J0_Conn1 pad K45: OAM0_S5_RX15N -> (no net)
- J0_Conn1 pad K46: OAM0_S5_RX15P -> (no net)
- J0_Conn1 pad K49: OAM0_S4_RX10N -> (no net)
- J0_Conn1 pad K5: OAM0_S7_RX15N -> (no net)
- J0_Conn1 pad K50: OAM0_S4_RX10P -> (no net)
- J0_Conn1 pad K53: OAM0_S4_RX13N -> (no net)
- J0_Conn1 pad K54: OAM0_S4_RX13P -> (no net)
- J0_Conn1 pad K57: OAM0_S4_RX15N -> (no net)
- J0_Conn1 pad K58: OAM0_S4_RX15P -> (no net)
- J0_Conn1 pad K6: OAM0_S7_RX15P -> (no net)
- J0_Conn1 pad K9: OAM0_S7_RX12N -> (no net)
- J0_Conn1 pad L11: OAM0_S7_RX11N -> (no net)
- J0_Conn1 pad L12: OAM0_S7_RX11P -> (no net)
- J0_Conn1 pad L15: OAM0_S7_RX9N -> (no net)
- J0_Conn1 pad L16: OAM0_S7_RX9P -> (no net)
- J0_Conn1 pad L19: OAM0_S6_RX8N -> (no net)
- J0_Conn1 pad L20: OAM0_S6_RX8P -> (no net)
- J0_Conn1 pad L23: OAM0_S6_RX10N -> (no net)
- J0_Conn1 pad L24: OAM0_S6_RX10P -> (no net)
- J0_Conn1 pad L27: OAM0_S6_RX12N -> (no net)
- J0_Conn1 pad L28: OAM0_S6_RX12P -> (no net)
- J0_Conn1 pad L3: OAM0_CONN2_INT# -> (no net)
- J0_Conn1 pad L31: OAM0_S6_RX14N -> (no net)
- J0_Conn1 pad L32: OAM0_S6_RX14P -> (no net)
- J0_Conn1 pad L35: OAM0_S5_RX9N -> (no net)
- J0_Conn1 pad L36: OAM0_S5_RX9P -> (no net)
- J0_Conn1 pad L39: OAM0_S5_RX11N -> (no net)
- J0_Conn1 pad L4: OAM0_CONN2_MODPRS# -> (no net)
- J0_Conn1 pad L40: OAM0_S5_RX11P -> (no net)
- J0_Conn1 pad L43: OAM0_S5_RX13N -> (no net)
- J0_Conn1 pad L44: OAM0_S5_RX13P -> (no net)
- J0_Conn1 pad L47: OAM0_S4_RX8N -> (no net)
- J0_Conn1 pad L48: OAM0_S4_RX8P -> (no net)
- J0_Conn1 pad L51: OAM0_S4_RX11N -> (no net)
- J0_Conn1 pad L52: OAM0_S4_RX11P -> (no net)
- J0_Conn1 pad L55: OAM0_S4_RX14N -> (no net)
- J0_Conn1 pad L56: OAM0_S4_RX14P -> (no net)
- J0_Conn1 pad L7: OAM0_S7_RX14N -> (no net)
- J0_Conn1 pad L8: OAM0_S7_RX14P -> (no net)
- J1_Conn0 pad A11: OAM1_S1_RX10P -> (no net)
- J1_Conn0 pad A12: OAM1_S1_RX10N -> (no net)
- J1_Conn0 pad A15: OAM1_S1_RX8P -> (no net)
- J1_Conn0 pad A16: OAM1_S1_RX8N -> (no net)
- J1_Conn0 pad A19: OAM1_S2_RX13P -> (no net)
- J1_Conn0 pad A20: OAM1_S2_RX13N -> (no net)
- J1_Conn0 pad A23: OAM1_S2_RX11P -> (no net)
- J1_Conn0 pad A24: OAM1_S2_RX11N -> (no net)
- J1_Conn0 pad A27: OAM1_S2_RX9P -> (no net)
- J1_Conn0 pad A28: OAM1_S2_RX9N -> (no net)
- J1_Conn0 pad A31: OAM1_S3_RX14P -> (no net)
- J1_Conn0 pad A32: OAM1_S3_RX14N -> (no net)
- J1_Conn0 pad A35: OAM1_S3_RX11P -> (no net)
- J1_Conn0 pad A36: OAM1_S3_RX11N -> (no net)
- J1_Conn0 pad A39: OAM1_S3_RX9P -> (no net)
- J1_Conn0 pad A40: OAM1_S3_RX9N -> (no net)
- J1_Conn0 pad A7: OAM1_S1_RX13P -> (no net)
- J1_Conn0 pad A8: OAM1_S1_RX13N -> (no net)
- J1_Conn0 pad B10: OAM1_S1_RX12N -> (no net)
- J1_Conn0 pad B13: OAM1_S1_RX9P -> (no net)
- J1_Conn0 pad B14: OAM1_S1_RX9N -> (no net)
- J1_Conn0 pad B17: OAM1_S2_RX15P -> (no net)
- J1_Conn0 pad B18: OAM1_S2_RX15N -> (no net)
- J1_Conn0 pad B21: OAM1_S2_RX12P -> (no net)
- J1_Conn0 pad B22: OAM1_S2_RX12N -> (no net)
- J1_Conn0 pad B25: OAM1_S2_RX10P -> (no net)
- J1_Conn0 pad B26: OAM1_S2_RX10N -> (no net)
- J1_Conn0 pad B29: OAM1_S2_RX8P -> (no net)
- J1_Conn0 pad B30: OAM1_S2_RX8N -> (no net)
- J1_Conn0 pad B33: OAM1_S3_RX13P -> (no net)
- J1_Conn0 pad B34: OAM1_S3_RX13N -> (no net)
- J1_Conn0 pad B37: OAM1_S3_RX10P -> (no net)
- J1_Conn0 pad B38: OAM1_S3_RX10N -> (no net)
- J1_Conn0 pad B41: OAM1_S3_RX8P -> (no net)
- J1_Conn0 pad B42: OAM1_S3_RX8N -> (no net)
- J1_Conn0 pad B5: OAM1_S1_RX15P -> (no net)
- J1_Conn0 pad B6: OAM1_S1_RX15N -> (no net)
- J1_Conn0 pad B9: OAM1_S1_RX12P -> (no net)
- J1_Conn0 pad C11: OAM1_S1_RX11P -> (no net)
- J1_Conn0 pad C12: OAM1_S1_RX11N -> (no net)
- J1_Conn0 pad C15: OAM1_S1_RX1P -> (no net)
- J1_Conn0 pad C16: OAM1_S1_RX1N -> (no net)
- J1_Conn0 pad C19: OAM1_S2_RX14P -> (no net)
- J1_Conn0 pad C20: OAM1_S2_RX14N -> (no net)
- J1_Conn0 pad C23: OAM1_S2_RX4P -> (no net)
- J1_Conn0 pad C24: OAM1_S2_RX4N -> (no net)
- J1_Conn0 pad C27: OAM1_S2_RX1P -> (no net)
- J1_Conn0 pad C28: OAM1_S2_RX1N -> (no net)
- J1_Conn0 pad C31: OAM1_S3_RX15P -> (no net)
- J1_Conn0 pad C32: OAM1_S3_RX15N -> (no net)
- J1_Conn0 pad C35: OAM1_S3_RX12P -> (no net)
- J1_Conn0 pad C36: OAM1_S3_RX12N -> (no net)
- J1_Conn0 pad C39: OAM1_S3_RX2P -> (no net)
- J1_Conn0 pad C40: OAM1_S3_RX2N -> (no net)
- J1_Conn0 pad C7: OAM1_S1_RX14P -> (no net)
- J1_Conn0 pad C8: OAM1_S1_RX14N -> (no net)
- J1_Conn0 pad D10: OAM1_S1_RX5N -> (no net)
- J1_Conn0 pad D13: OAM1_S1_RX3P -> (no net)
- J1_Conn0 pad D14: OAM1_S1_RX3N -> (no net)
- J1_Conn0 pad D17: OAM1_S1_RX0P -> (no net)
- J1_Conn0 pad D18: OAM1_S1_RX0N -> (no net)
- J1_Conn0 pad D21: OAM1_S2_RX6P -> (no net)
- J1_Conn0 pad D22: OAM1_S2_RX6N -> (no net)
- J1_Conn0 pad D25: OAM1_S2_RX3P -> (no net)
- J1_Conn0 pad D26: OAM1_S2_RX3N -> (no net)
- J1_Conn0 pad D29: OAM1_S2_RX0P -> (no net)
- J1_Conn0 pad D30: OAM1_S2_RX0N -> (no net)
- J1_Conn0 pad D33: OAM1_S3_RX6P -> (no net)
- J1_Conn0 pad D34: OAM1_S3_RX6N -> (no net)
- J1_Conn0 pad D37: OAM1_S3_RX4P -> (no net)
- J1_Conn0 pad D38: OAM1_S3_RX4N -> (no net)
- J1_Conn0 pad D41: OAM1_S3_RX1P -> (no net)
- J1_Conn0 pad D42: OAM1_S3_RX1N -> (no net)
- J1_Conn0 pad D5: OAM1_S1_RX7P -> (no net)
- J1_Conn0 pad D6: OAM1_S1_RX7N -> (no net)
- J1_Conn0 pad D9: OAM1_S1_RX5P -> (no net)
- J1_Conn0 pad E11: OAM1_S1_RX4P -> (no net)
- J1_Conn0 pad E12: OAM1_S1_RX4N -> (no net)
- J1_Conn0 pad E15: OAM1_S1_RX2P -> (no net)
- J1_Conn0 pad E16: OAM1_S1_RX2N -> (no net)
- J1_Conn0 pad E19: OAM1_S2_RX7P -> (no net)
- J1_Conn0 pad E20: OAM1_S2_RX7N -> (no net)
- J1_Conn0 pad E23: OAM1_S2_RX5P -> (no net)
- J1_Conn0 pad E24: OAM1_S2_RX5N -> (no net)
- J1_Conn0 pad E27: OAM1_S2_RX2P -> (no net)
- J1_Conn0 pad E28: OAM1_S2_RX2N -> (no net)
- J1_Conn0 pad E31: OAM1_S3_RX7P -> (no net)
- J1_Conn0 pad E32: OAM1_S3_RX7N -> (no net)
- J1_Conn0 pad E35: OAM1_S3_RX5P -> (no net)
- J1_Conn0 pad E36: OAM1_S3_RX5N -> (no net)
- J1_Conn0 pad E39: OAM1_S3_RX3P -> (no net)
- J1_Conn0 pad E40: OAM1_S3_RX3N -> (no net)
- J1_Conn0 pad E43: OAM1_S3_RX0P -> (no net)
- J1_Conn0 pad E44: OAM1_S3_RX0N -> (no net)
- J1_Conn0 pad E7: OAM1_S1_RX6P -> (no net)
- J1_Conn0 pad E8: OAM1_S1_RX6N -> (no net)
- J1_Conn0 pad G11: OAM1_S1_TX10P -> (no net)
- J1_Conn0 pad G12: OAM1_S1_TX10N -> (no net)
- J1_Conn0 pad G15: OAM1_S1_TX8P -> (no net)
- J1_Conn0 pad G16: OAM1_S1_TX8N -> (no net)
- J1_Conn0 pad G19: OAM1_S2_TX13P -> (no net)
- J1_Conn0 pad G20: OAM1_S2_TX13N -> (no net)
- J1_Conn0 pad G23: OAM1_S2_TX11P -> (no net)
- J1_Conn0 pad G24: OAM1_S2_TX11N -> (no net)
- J1_Conn0 pad G27: OAM1_S2_TX9P -> (no net)
- J1_Conn0 pad G28: OAM1_S2_TX9N -> (no net)
- J1_Conn0 pad G31: OAM1_S3_TX14P -> (no net)
- J1_Conn0 pad G32: OAM1_S3_TX14N -> (no net)
- J1_Conn0 pad G35: OAM1_S3_TX12P -> (no net)
- J1_Conn0 pad G36: OAM1_S3_TX12N -> (no net)
- J1_Conn0 pad G39: OAM1_S3_TX10P -> (no net)
- J1_Conn0 pad G40: OAM1_S3_TX10N -> (no net)
- J1_Conn0 pad G43: OAM1_S3_TX8P -> (no net)
- J1_Conn0 pad G44: OAM1_S3_TX8N -> (no net)
- J1_Conn0 pad G7: OAM1_S1_TX13P -> (no net)
- J1_Conn0 pad G8: OAM1_S1_TX13N -> (no net)
- J1_Conn0 pad H10: OAM1_S1_TX12N -> (no net)
- J1_Conn0 pad H13: OAM1_S1_TX9P -> (no net)
- J1_Conn0 pad H14: OAM1_S1_TX9N -> (no net)
- J1_Conn0 pad H17: OAM1_S2_TX15P -> (no net)
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Routing:
- added copper zone on In1.Cu, net GND
- added copper zone on In10.Cu, net GND
- added copper zone on In4.Cu, net GND
- added copper zone on In7.Cu, net GND
- added copper zone on F.Cu, net P48V
- added copper zone on F.Cu, net P48V_STAR
Other:
- copper layers 4 -> 12
- board text added: "12L 2.0mm stuffed-switch TARGET. 8L 2.0mm is cheaper DNP option only. No signal tracks yet."
- board text added: "3x x16 + 4x x8 Gen3 MPN Unknown"
- board text added: "HOST CABLE KEEPOUT"
- board text added: "Molex 218910-1115 x16 | 12L 2.0mm TARGET | LOCAL P48V pours | 2x PM8536B-FEI DNP | SB175 star | NOT a UBB"
- board text added: "P12V1 in <=50W MPN Unknown no VRM"
- board text added: "P12V2 pads named v1.0 — Unknown / may be NC — do not short to P12V1"
- board text added: "P3V3 in <=5W MPN Unknown no VRM"
- board text added: "P48V STAR / Kelvin sense"
- board text added: "P48V local pour — 16 Conn0 pads — 2 oz — not a 100A plane"
- board text added: "PM8536B-FEI 37.5mm 1311-FCBGA"
- board text added: "SEAT 0 ELEC NAMED first-stuff OK PE->SW0 x8/GCD"
- board text added: "SEAT 1 ELEC NAMED first-stuff OK PE->SW0 x8/GCD"
- board text added: "SEAT 2 ELEC NAMED module DNP OK PE->SW0 no respin"
- board text added: "SEAT 3 ELEC NAMED module DNP OK PE->SW0 no respin"
- board text added: "SEAT 4 ELEC NAMED module DNP OK PE->SW1 no respin"
- board text added: "SEAT 5 ELEC NAMED module DNP OK PE->SW1 no respin"
- board text added: "SEAT 6 ELEC NAMED module DNP OK PE->SW1 no respin"
- board text added: "SEAT 7 ELEC NAMED module DNP OK PE->SW1 no respin"
- board text added: "STAR-FED P48V — LOCAL POURS ONLY — DO NOT ENERGIZE"
- board text added: "U_SW0 DNP"
- board text added: "U_SW1 DNP"
- board text added: "X11DPH-T two CPU x16 uplinks"
- board text added: "off-board 48V via 2 AWG | NOT D3000E-S1 12V"
- board text added: "seats 0-3 x8/GCD 16US+64DS"
- board text added: "seats 4-7 x8/GCD 16US+64DS"
- board text added: "~15A FUSE S0 MPN Unknown"
- board text added: "~15A FUSE S1 MPN Unknown"
- board text added: "~15A FUSE S2 MPN Unknown"
- board text added: "~15A FUSE S3 MPN Unknown"
- board text added: "~15A FUSE S4 MPN Unknown"
- board text added: "~15A FUSE S5 MPN Unknown"
- board text added: "~15A FUSE S6 MPN Unknown"
- board text added: "~15A FUSE S7 MPN Unknown"
- board text removed: "HOST CONNECTOR REGION"
- board text removed: "Inners In1.Cu / In2.Cu reserved. No signal tracks. Seats 2-7 have power nets only."
- board text removed: "Molex 218910-1115 x16 | 4-layer | no P48V pour | ticket 167157 | NOT a UBB"
- board text removed: "OAM0+OAM1 PCIE_* named nets point here"
- board text removed: "P48V PADS EXIST — NO POUR — DO NOT ENERGIZE"
- board text removed: "SEAT 0 HOST PCIe NAMED (stub) populate now"
- board text removed: "SEAT 1 HOST PCIe NAMED (stub) populate now"
- board text removed: "SEAT 2 MECH+POWER ONLY needs on-board PCIe switch — MPN Unknown"
- board text removed: "SEAT 3 MECH+POWER ONLY needs on-board PCIe switch — MPN Unknown"
- board text removed: "SEAT 4 MECH+POWER ONLY needs on-board PCIe switch — MPN Unknown"
- board text removed: "SEAT 5 MECH+POWER ONLY needs on-board PCIe switch — MPN Unknown"
- board text removed: "SEAT 6 MECH+POWER ONLY needs on-board PCIe switch — MPN Unknown"
- board text removed: "SEAT 7 MECH+POWER ONLY needs on-board PCIe switch — MPN Unknown"
- board text removed: "seats 2-7: needs on-board PCIe switch — MPN Unknown"

Commit message: Label PEX8780-AB80BI G as the only switch CANDIDATE (DNP).
Keepout is one 35 mm 1156-FCBGA for 8x x8 Gen3 plus one x16 host uplink.
Do not invent a second MPN. Do not stuff. 8-layer is likely if this BGA
is ever assembled; PCBWay 1156-FCBGA attach remains Unknown.

Still do not fabricate or energize P48V. No xGMI, no CEM.

Co-authored-by: zivzancoeli-commits <zivzancoeli-commits@users.noreply.github.com>
Other:
- board text added: "35mm 1156-FCBGA 80-lane"
- board text added: "8x x8 + one x16 UL NOT stuffed"
- board text added: "Molex 218910-1115 x16 | PEX8780-AB80BI G CANDIDATE DNP | 8L likely if stuffed | SB175 star | NOT a UBB"
- board text added: "NO SECOND SWITCH MPN"
- board text added: "PEX8780 CANDIDATE DNP. 8L likely if 1156 stuffed. PCBWay 1156 assembly Unknown. No signal tracks."
- board text added: "PEX8780-AB80BI G"
- board text added: "PEX8796 / PEX88096 / PM40100 not placed"
- board text added: "SEAT 0 ELEC NAMED first-stuff OK PE->PEX8780 x8"
- board text added: "SEAT 1 ELEC NAMED first-stuff OK PE->PEX8780 x8"
- board text added: "SEAT 2 ELEC NAMED module DNP OK PE->PEX8780 x8 no respin"
- board text added: "SEAT 3 ELEC NAMED module DNP OK PE->PEX8780 x8 no respin"
- board text added: "SEAT 4 ELEC NAMED module DNP OK PE->PEX8780 x8 no respin"
- board text added: "SEAT 5 ELEC NAMED module DNP OK PE->PEX8780 x8 no respin"
- board text added: "SEAT 6 ELEC NAMED module DNP OK PE->PEX8780 x8 no respin"
- board text added: "SEAT 7 ELEC NAMED module DNP OK PE->PEX8780 x8 no respin"
- board text added: "U_SW CANDIDATE DNP"
- board text added: "X11DPH-T one CPU x16 uplink"
- board text removed: "12L 2.0mm stuffed-switch TARGET. 8L 2.0mm is cheaper DNP option only. No signal tracks yet."
- board text removed: "Molex 218910-1115 x16 | 12L 2.0mm TARGET | LOCAL P48V pours | 2x PM8536B-FEI DNP | SB175 star | NOT a UBB"
- board text removed: "PM8536B-FEI 37.5mm 1311-FCBGA"
- board text removed: "SEAT 0 ELEC NAMED first-stuff OK PE->SW0 x8/GCD"
- board text removed: "SEAT 1 ELEC NAMED first-stuff OK PE->SW0 x8/GCD"
- board text removed: "SEAT 2 ELEC NAMED module DNP OK PE->SW0 no respin"
- board text removed: "SEAT 3 ELEC NAMED module DNP OK PE->SW0 no respin"
- board text removed: "SEAT 4 ELEC NAMED module DNP OK PE->SW1 no respin"
- board text removed: "SEAT 5 ELEC NAMED module DNP OK PE->SW1 no respin"
- board text removed: "SEAT 6 ELEC NAMED module DNP OK PE->SW1 no respin"
- board text removed: "SEAT 7 ELEC NAMED module DNP OK PE->SW1 no respin"
- board text removed: "U_SW0 DNP"
- board text removed: "U_SW1 DNP"
- board text removed: "X11DPH-T two CPU x16 uplinks"
- board text removed: "seats 0-3 x8/GCD 16US+64DS"
- board text removed: "seats 4-7 x8/GCD 16US+64DS"
Changed lines of the file:
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@@
     (rev "Rev3_8Seat_PCBWay_v1")
     (comment 1 "DO NOT FABRICATE. DO NOT ENERGIZE P48V. Molex 60V written; 1.2A/contact OPEN.")
-    (comment 2 "492 x 372 mm 12-layer 2.0 mm stuffed-switch TARGET. Local P48V. 2x PM8536 DNP. SB175.")
+    (comment 2 "492 x 372 mm. PEX8780-AB80BI G CANDIDATE DNP. 8L likely if stuffed. SB175.")
   )
   (layers
@@
     (at 246.000 6) (layer "F.SilkS")
     (effects (font (size 2.4 2.4) (thickness 0.3))))
-  (gr_text "Molex 218910-1115 x16  |  12L 2.0mm TARGET  |  LOCAL P48V pours  |  2x PM8536B-FEI DNP  |  SB175 star  |  NOT a UBB"
+  (gr_text "Molex 218910-1115 x16  |  PEX8780-AB80BI G CANDIDATE DNP  |  8L likely if stuffed  |  SB175 star  |  NOT a UBB"
     (at 246.000 12) (layer "F.SilkS")
     (effects (font (size 1.5 1.5) (thickness 0.18))))
@@
   (gr_rect (start 20.500 20.500) (end 122.500 185.500)
     (stroke (width 0.12) (type dash)) (fill none) (layer "Dwgs.User"))
-  (gr_text "SEAT 0  ELEC NAMED  first-stuff OK  PE->SW0  x8/GCD"
+  (gr_text "SEAT 0  ELEC NAMED  first-stuff OK  PE->PEX8780  x8"
     (at 71.500 28.000) (layer "F.SilkS")
     (effects (font (size 1.5 1.5) (thickness 0.18))))
@@
   (gr_rect (start 123.500 20.500) (end 225.500 185.500)
     (stroke (width 0.12) (type dash)) (fill none) (layer "Dwgs.User"))
-  (gr_text "SEAT 1  ELEC NAMED  first-stuff OK  PE->SW0  x8/GCD"
+  (gr_text "SEAT 1  ELEC NAMED  first-stuff OK  PE->PEX8780  x8"
     (at 174.500 28.000) (layer "F.SilkS")
     (effects (font (size 1.5 1.5) (thickness 0.18))))
@@
   (gr_rect (start 226.500 20.500) (end 328.500 185.500)
     (stroke (width 0.12) (type dash)) (fill none) (layer "Dwgs.User"))
-  (gr_text "SEAT 2  ELEC NAMED  module DNP OK  PE->SW0  no respin"
+  (gr_text "SEAT 2  ELEC NAMED  module DNP OK  PE->PEX8780  x8  no respin"
     (at 277.500 28.000) (layer "F.SilkS")
     (effects (font (size 1.5 1.5) (thickness 0.18))))
@@
   (gr_rect (start 329.500 20.500) (end 431.500 185.500)
     (stroke (width 0.12) (type dash)) (fill none) (layer "Dwgs.User"))
-  (gr_text "SEAT 3  ELEC NAMED  module DNP OK  PE->SW0  no respin"
+  (gr_text "SEAT 3  ELEC NAMED  module DNP OK  PE->PEX8780  x8  no respin"
     (at 380.500 28.000) (layer "F.SilkS")
     (effects (font (size 1.5 1.5) (thickness 0.18))))
@@
   (gr_rect (start 20.500 186.500) (end 122.500 351.500)
     (stroke (width 0.12) (type dash)) (fill none) (layer "Dwgs.User"))
-  (gr_text "SEAT 4  ELEC NAMED  module DNP OK  PE->SW1  no respin"
+  (gr_text "SEAT 4  ELEC NAMED  module DNP OK  PE->PEX8780  x8  no respin"
     (at 71.500 194.000) (layer "F.SilkS")
     (effects (font (size 1.5 1.5) (thickness 0.18))))
@@
   (gr_rect (start 123.500 186.500) (end 225.500 351.500)
     (stroke (width 0.12) (type dash)) (fill none) (layer "Dwgs.User"))
-  (gr_text "SEAT 5  ELEC NAMED  module DNP OK  PE->SW1  no respin"
+  (gr_text "SEAT 5  ELEC NAMED  module DNP OK  PE->PEX8780  x8  no respin"
     (at 174.500 194.000) (layer "F.SilkS")
     (effects (font (size 1.5 1.5) (thickness 0.18))))
@@
   (gr_rect (start 226.500 186.500) (end 328.500 351.500)
     (stroke (width 0.12) (type dash)) (fill none) (layer "Dwgs.User"))
-  (gr_text "SEAT 6  ELEC NAMED  module DNP OK  PE->SW1  no respin"
+  (gr_text "SEAT 6  ELEC NAMED  module DNP OK  PE->PEX8780  x8  no respin"
     (at 277.500 194.000) (layer "F.SilkS")
     (effects (font (size 1.5 1.5) (thickness 0.18))))
@@
   (gr_rect (start 329.500 186.500) (end 431.500 351.500)
     (stroke (width 0.12) (type dash)) (fill none) (layer "Dwgs.User"))
-  (gr_text "SEAT 7  ELEC NAMED  module DNP OK  PE->SW1  no respin"
+  (gr_text "SEAT 7  ELEC NAMED  module DNP OK  PE->PEX8780  x8  no respin"
     (at 380.500 194.000) (layer "F.SilkS")
     (effects (font (size 1.5 1.5) (thickness 0.18))))
@@
   (gr_rect (start 452.000 28.000) (end 492.000 68.000)
     (stroke (width 0.2) (type dash)) (fill none) (layer "Dwgs.User"))
-  (gr_text "U_SW0 DNP"
+  (gr_text "U_SW CANDIDATE DNP"
     (at 472.000 48.000 90) (layer "F.SilkS")
-    (effects (font (size 1.4 1.4) (thickness 0.16))))
-  (gr_text "PM8536B-FEI 37.5mm 1311-FCBGA"
+    (effects (font (size 1.3 1.3) (thickness 0.16))))
+  (gr_text "PEX8780-AB80BI G"
     (at 480.000 48.000 90) (layer "F.SilkS")
-    (effects (font (size 1.0 1.0) (thickness 0.12))))
-  (gr_text "seats 0-3  x8/GCD  16US+64DS"
+    (effects (font (size 1.1 1.1) (thickness 0.14))))
+  (gr_text "35mm 1156-FCBGA  80-lane"
     (at 488.000 48.000 90) (layer "F.SilkS")
     (effects (font (size 0.9 0.9) (thickness 0.1))))
+  (gr_text "8x x8 + one x16 UL  NOT stuffed"
+    (at 496.000 48.000 90) (layer "F.SilkS")
+    (effects (font (size 0.85 0.85) (thickness 0.1))))
   (gr_rect (start 452.000 90.000) (end 492.000 250.000)
     (stroke (width 0.2) (type dash)) (fill none) (layer "F.CrtYd"))
@@
     (at 472.000 170.000 90) (layer "F.SilkS")
     (effects (font (size 1.5 1.5) (thickness 0.18))))
-  (gr_text "X11DPH-T two CPU x16 uplinks"
+  (gr_text "X11DPH-T one CPU x16 uplink"
     (at 464.000 170.000 90) (layer "F.SilkS")
     (effects (font (size 1.1 1.1) (thickness 0.14))))
@@
     (at 488.000 170.000 90) (layer "F.SilkS")
     (effects (font (size 1.1 1.1) (thickness 0.14))))
-  (gr_rect (start 452.000 284.000) (end 492.000 324.000)
-    (stroke (width 0.25) (type dash)) (fill none) (layer "F.CrtYd"))
-  (gr_rect (start 452.000 284.000) (end 492.000 324.000)
-    (stroke (width 0.2) (type dash)) (fill none) (layer "Dwgs.User"))
-  (gr_text "U_SW1 DNP"
+  (gr_text "NO SECOND SWITCH MPN"
     (at 472.000 304.000 90) (layer "F.SilkS")
-    (effects (font (size 1.4 1.4) (thickness 0.16))))
-  (gr_text "PM8536B-FEI 37.5mm 1311-FCBGA"
-    (at 480.000 304.000 90) (layer "F.SilkS")
-    (effects (font (size 1.0 1.0) (thickness 0.12))))
-  (gr_text "seats 4-7  x8/GCD  16US+64DS"
-    (at 488.000 304.000 90) (layer "F.SilkS")
-    (effects (font (size 0.9 0.9) (thickness 0.1))))
+    (effects (font (size 1.2 1.2) (thickness 0.14))))
+  (gr_text "PEX8796 / PEX88096 / PM40100 not placed"
+    (at 482.000 304.000 90) (layer "F.SilkS")
+    (effects (font (size 0.85 0.85) (thickness 0.1))))
   (gr_text "STAR-FED P48V — LOCAL POURS ONLY — DO NOT ENERGIZE"
     (at 246.000 360.000) (layer "F.SilkS")
     (effects (font (size 1.8 1.8) (thickness 0.22))))
-  (gr_text "12L 2.0mm stuffed-switch TARGET. 8L 2.0mm is cheaper DNP option only. No signal tracks yet."
+  (gr_text "PEX8780 CANDIDATE DNP. 8L likely if 1156 stuffed. PCBWay 1156 assembly Unknown. No signal tracks."
     (at 246.000 16.5) (layer "Cmts.User")
     (effects (font (size 1.2 1.2) (thickness 0.14))))
@@
   )
   (zone (net 0) (net_name "") (layers "*.Cu")
-    (hatch edge 0.5)
-    (priority 0)
-    (keepout (tracks not_allowed) (vias not_allowed) (pads allowed) (copperpour not_allowed) (footprints not_allowed))
-    (fill yes (thermal_gap 0.5) (thermal_bridge_width 0.5))
-    (polygon (pts (xy 452.000 284.000) (xy 492.000 284.000) (xy 492.000 324.000) (xy 452.000 324.000)))
-  )
-  (zone (net 0) (net_name "") (layers "*.Cu")
