File: Generated_Project/Rev3_8Seat_PCBWay_Chassis_v1/MI250X_8OAM_PCBWay_Chassis_Stub.kicad_pcb (KiCad board)
At the start: 12 copper layers, 492 x 372 mm, 60 parts, among them J0_Conn0 218910-1115, J0_Conn1 218910-1115, J1_Conn0 218910-1115, J1_Conn1 218910-1115, J2_Conn0 218910-1115, J2_Conn1 218910-1115, J3_Conn0 218910-1115, J3_Conn1 218910-1115, J4_Conn0 218910-1115, J4_Conn1 218910-1115, J5_Conn0 218910-1115, J5_Conn1 218910-1115, J6_Conn0 218910-1115, J6_Conn1 218910-1115, J7_Conn0 218910-1115, J7_Conn1 218910-1115

Commit message: Document an 8x full-width chassis CONCEPT (ideas only, not fab).
Sibling folder plus STATUS pointer. Comments-layer KiCad notes say
CONCEPT / DO NOT FABRICATE. No overlay, ball map, CEM/MCIO, r2.0, or
S1-S7 assignment. X11DPH-T cannot light 256 DS. Do not energize.
Do not upload to PCBWay.

Co-authored-by: zivzancoeli-commits <zivzancoeli-commits@users.noreply.github.com>
Other:
- board text added: "CONCEPT 8x FULL-WIDTH: see Rev3_8Seat_FULLWIDTH_CONCEPT/CONCEPT.md — DO NOT FABRICATE as live PE. X11DPH-T cannot light 256 DS. GCD1 named-only. xGMI=XGMI_Sn_P* boxes only, not S1-S7."
Changed lines of the file:
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@@
+		)
+	)
+	(gr_text "CONCEPT 8x FULL-WIDTH: see Rev3_8Seat_FULLWIDTH_CONCEPT/CONCEPT.md — DO NOT FABRICATE as live PE. X11DPH-T cannot light 256 DS. GCD1 named-only. xGMI=XGMI_Sn_P* boxes only, not S1-S7."
+		(at 246 346 0)
+		(layer "Cmts.User")
+		(effects
+			(font
+				(size 1.0 1.0)
+				(thickness 0.12)
+			)
 		)
 	)
