File: Generated_Project/Rev3_8Seat_PCBWay_Chassis_v1/MI250X_8OAM_PCBWay_Chassis_Stub.kicad_pcb (KiCad board)
At the start: 12 copper layers, 492 x 372 mm, 60 parts, among them J0_Conn0 218910-1115, J0_Conn1 218910-1115, J1_Conn0 218910-1115, J1_Conn1 218910-1115, J2_Conn0 218910-1115, J2_Conn1 218910-1115, J3_Conn0 218910-1115, J3_Conn1 218910-1115, J4_Conn0 218910-1115, J4_Conn1 218910-1115, J5_Conn0 218910-1115, J5_Conn1 218910-1115, J6_Conn0 218910-1115, J6_Conn1 218910-1115, J7_Conn0 218910-1115, J7_Conn1 218910-1115

Commit message: Reserve late-bind hooks; 16x x16 PE remains a copper respin.
Document what overlay, PM8536, host plug, Molex 1.2 A, and cooling
already have vs what a later spin must add. Comment-layer corridors
for seats 0-1 GCD0 toward host keepout and SW0; no guessed tracks.
Do not claim the POWER+MECH zip works as a live GPU chassis.
Do not energize. Do not upload to PCBWay.

Co-authored-by: zivzancoeli-commits <zivzancoeli-commits@users.noreply.github.com>
Other:
- board text added: "LATE BIND note: PE_S0/S1_GCD0 toward SW0 courtyard. NO COPPER. 1311-ball escape = RESPIN. See LATE_BIND.md."
- board text added: "LATE BIND note: PE_S0/S1_GCD0 toward host keepout. NO COPPER. NO FAKE PINS. 16x x16 route = RESPIN not silk ECO."
Changed lines of the file:
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@@
+		)
+	)
+	(gr_rect
+		(start 105 138)
+		(end 452 178)
+		(stroke
+			(width 0.18)
+			(type dash)
+		)
+		(fill none)
+		(layer "Dwgs.User")
+	)
+	(gr_text "LATE BIND note: PE_S0/S1_GCD0 toward host keepout. NO COPPER. NO FAKE PINS. 16x x16 route = RESPIN not silk ECO."
+		(at 278.5 158 0)
+		(layer "Cmts.User")
+		(effects
+			(font
+				(size 0.9 0.9)
+				(thickness 0.1)
+			)
+		)
+	)
+	(gr_rect
+		(start 105 22)
+		(end 452 56)
+		(stroke
+			(width 0.18)
+			(type dash)
+		)
+		(fill none)
+		(layer "Dwgs.User")
+	)
+	(gr_text "LATE BIND note: PE_S0/S1_GCD0 toward SW0 courtyard. NO COPPER. 1311-ball escape = RESPIN. See LATE_BIND.md."
+		(at 278.5 39 0)
+		(layer "Cmts.User")
+		(effects
+			(font
+				(size 0.9 0.9)
+				(thickness 0.1)
+			)
 		)
 	)
