File: Generated_Project/Rev3_8Seat_PCBWay_Chassis_v1/MI250X_8OAM_PCBWay_Chassis_Stub.kicad_sch (KiCad schematic)
At the start: 0 parts

Commit message: Raise Rev3 chassis to 8 electrically designed seats.
Name v1.0 power/PE/clock nets on all eight OAM seats toward two DNP
PM8536B-FEI (x8 per GCD), keep SB175 star + local P48V pours, and generate
the 12-layer 2.0 mm stuffed-switch target. First stuffing may still populate
two modules; the PCB does not need a respin for the other six.

Do not fabricate. Do not energize P48V.

Co-authored-by: zivzancoeli-commits <zivzancoeli-commits@users.noreply.github.com>
Other:
- removed sheet 11_PCIe_Switch_Unknown
- added sheet 11_PM8536_DNP (sheets/11_pcie_switch_unknown.kicad_sch)
- note added: "DO NOT FABRICATE / DO NOT ENERGIZE P48V 8 electrically designed OAM seats (first stuffing: 2 modules / 6 DNP OK — no respin). 16x Molex 218910-1115, 5.00 mm stack. 12-layer 2.0 mm stuffed-switch TARGET. Outline 492 x 372 mm. 4x2 of 103x166 mm KOZ = 412x332 mm INFERRED tiling (not a UBB drawing). All 8: named PE toward 2x PM8536B-FEI DNP (x8/GCD; SW0=0-3, SW1=4-7). No CEM invented. Host stub: X11D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"
- note removed: "DO NOT FABRICATE / DO NOT ENERGIZE P48V 8 identical OAM seats (populate 0-1 now, 2-7 later). Same board. 16x Molex 218910-1115, 5.00 mm stack. 4-layer FR-4. Outline 492 x 372 mm. 4x2 of 103x166 mm KOZ = 412x332 mm INFERRED tiling (not a UBB drawing). Seats 0-1: named host PCIe nets toward HOST CONNECTOR REGION. No CEM invented. Seats 2-7: mechanical+power only. needs on-board PCIe switch — MPN Un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"
Changed lines of the file:
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@@
 		(date "2026-08-21")
 		(rev "Rev3_8Seat_PCBWay_v1")
-		(comment 1 "DO NOT FABRICATE. DO NOT ENERGIZE P48V. Ticket 167157 open.")
-		(comment 2 "8 OAM seats. Host X11DPH-T is NOT on this PCB. No CEM cable. No 20-layer UBB.")
-		(comment 3 "Pin names: OAM Pin map rev 1.0.xlsx — OCP generic, NOT AMD overlay")
-		(comment 4 "r2.0 maps UNUSABLE. P3V3=2 Conn0 C1/C2. 8-seat PCBWay chassis stub.")
-	)
-	(text "DO NOT FABRICATE / DO NOT ENERGIZE P48V\n8 identical OAM seats (populate 0-1 now, 2-7 later). Same board.\n16x Molex 218910-1115, 5.00 mm stack. 4-layer FR-4. Outline 492 x 372 mm.\n4x2 of 103x166 mm KOZ = 412x332 mm INFERRED tiling (not a UBB drawing).\nSeats 0-1: named host PCIe nets toward HOST CONNECTOR REGION. No CEM invented.\nSeats 2-7: mechanical+power only. needs on-board PCIe switch — MPN Unknown.\nX11DPH-T: 3x Gen3 x16 + 4x Gen3 x8. NOT enough lanes for 8x MI250X (2 GCD, typically 2x x16).\nS1-S7 NOT routed between OAMs. TEST*/RFU/DO_NOT_USE unmapped. PVREF never driven.\nP48V pads exist, NO POUR. Molex catalog 30 V vs OCP 44-59.5 V, ticket 167157.\nDell D3000E-S1 is 12 V CRPS — do not mix. P3V3 = Conn0 C1/C2 only. Never r2.0."
+        (comment 1 "DO NOT FABRICATE. DO NOT ENERGIZE P48V. Molex 60V written 2026-08-18; 1.2A/contact OPEN.")
+        (comment 2 "8 OAM seats. Host X11DPH-T is NOT on this PCB. No CEM cable. No 20-layer UBB.")
+        (comment 3 "Pin names: OAM Pin map rev 1.0.xlsx — OCP generic, NOT AMD overlay")
+        (comment 4 "r2.0 UNUSABLE. P3V3=Conn0 C1/C2. 12L 2.0mm stuffed-switch TARGET. Star-fed P48V.")
+	)
+	(text "DO NOT FABRICATE / DO NOT ENERGIZE P48V\n8 electrically designed OAM seats (first stuffing: 2 modules / 6 DNP OK — no respin).\n16x Molex 218910-1115, 5.00 mm stack. 12-layer 2.0 mm stuffed-switch TARGET. Outline 492 x 372 mm.\n4x2 of 103x166 mm KOZ = 412x332 mm INFERRED tiling (not a UBB drawing).\nAll 8: named PE toward 2x PM8536B-FEI DNP (x8/GCD; SW0=0-3, SW1=4-7). No CEM invented.\nHost stub: X11DPH-T 3x Gen3 x16 + 4x Gen3 x8 keepout. Two CPU x16 = switch uplinks.\nX11DPH-T / NH-D9 DX-3647 / B550M are NOT on this PCB. Chamber A mATX is not this PCB.\nS1-S7 NOT routed (no xGMI). TEST*/RFU/DO_NOT_USE unmapped. PVREF never driven.\nP48V: SB175 long-edge entry + ~15A fuse/seat + LOCAL pours on 16 Conn0 pads. NOT a 100A flood.\nMolex 2026-08-18: CSA 60V (COFC 80170713) at OCP P48V; skip pins = published map, no extra NC.\nOPEN: 1.2 A/contact at 48-59.5 V (2 oz). HOST_PWRGD is ENABLE. No GPU VRM. P12V2 Unknown/may be NC.\nDell D3000E-S1 is 12 V CRPS — do not mix into P48V. P3V3 = Conn0 C1/C2 only. Never r2.0."
 		(exclude_from_sim no)
 		(at 25.4 15.24 0)
@@
 		(instances
 			(project "MI250X_8OAM_PCBWay_Chassis_Stub"
-				(path "/9e149b2c-ee24-41e4-9a2c-1616a441d16c"
+				(path "/037bf010-d9fb-4db9-9927-6079b8b745cf"
 					(page "2")
 				)
@@
 		(instances
 			(project "MI250X_8OAM_PCBWay_Chassis_Stub"
-				(path "/9e149b2c-ee24-41e4-9a2c-1616a441d16c"
+				(path "/037bf010-d9fb-4db9-9927-6079b8b745cf"
 					(page "3")
 				)
@@
 		(instances
 			(project "MI250X_8OAM_PCBWay_Chassis_Stub"
-				(path "/9e149b2c-ee24-41e4-9a2c-1616a441d16c"
+				(path "/037bf010-d9fb-4db9-9927-6079b8b745cf"
 					(page "4")
 				)
@@
 		(instances
 			(project "MI250X_8OAM_PCBWay_Chassis_Stub"
-				(path "/9e149b2c-ee24-41e4-9a2c-1616a441d16c"
+				(path "/037bf010-d9fb-4db9-9927-6079b8b745cf"
 					(page "5")
 				)
@@
 		(instances
 			(project "MI250X_8OAM_PCBWay_Chassis_Stub"
-				(path "/9e149b2c-ee24-41e4-9a2c-1616a441d16c"
+				(path "/037bf010-d9fb-4db9-9927-6079b8b745cf"
 					(page "6")
 				)
@@
 		(instances
 			(project "MI250X_8OAM_PCBWay_Chassis_Stub"
-				(path "/9e149b2c-ee24-41e4-9a2c-1616a441d16c"
+				(path "/037bf010-d9fb-4db9-9927-6079b8b745cf"
 					(page "7")
 				)
@@
 		(instances
 			(project "MI250X_8OAM_PCBWay_Chassis_Stub"
-				(path "/9e149b2c-ee24-41e4-9a2c-1616a441d16c"
+				(path "/037bf010-d9fb-4db9-9927-6079b8b745cf"
 					(page "8")
 				)
@@
 		(instances
 			(project "MI250X_8OAM_PCBWay_Chassis_Stub"
-				(path "/9e149b2c-ee24-41e4-9a2c-1616a441d16c"
+				(path "/037bf010-d9fb-4db9-9927-6079b8b745cf"
 					(page "9")
 				)
@@
 		(instances
 			(project "MI250X_8OAM_PCBWay_Chassis_Stub"
-				(path "/9e149b2c-ee24-41e4-9a2c-1616a441d16c"
+				(path "/037bf010-d9fb-4db9-9927-6079b8b745cf"
 					(page "10")
 				)
@@
 		(instances
 			(project "MI250X_8OAM_PCBWay_Chassis_Stub"
-				(path "/9e149b2c-ee24-41e4-9a2c-1616a441d16c"
+				(path "/037bf010-d9fb-4db9-9927-6079b8b745cf"
 					(page "11")
 				)
@@
 		(instances
 			(project "MI250X_8OAM_PCBWay_Chassis_Stub"
-				(path "/9e149b2c-ee24-41e4-9a2c-1616a441d16c"
+				(path "/037bf010-d9fb-4db9-9927-6079b8b745cf"
 					(page "12")
 				)
@@
 		(stroke (width 0.1524) (type solid))
 		(fill (color 0 0 0 0.0000))
-		(property "Sheetname" "11_PCIe_Switch_Unknown"
+		(property "Sheetname" "11_PM8536_DNP"
 			(at 238.54 181.46 0)
 			(effects (font (size 1.27 1.27)) (justify left bottom))
@@
 		(instances
 			(project "MI250X_8OAM_PCBWay_Chassis_Stub"
-				(path "/9e149b2c-ee24-41e4-9a2c-1616a441d16c"
+				(path "/037bf010-d9fb-4db9-9927-6079b8b745cf"
 					(page "13")
 				)
@@
 		(instances
 			(project "MI250X_8OAM_PCBWay_Chassis_Stub"
-				(path "/9e149b2c-ee24-41e4-9a2c-1616a441d16c"
+				(path "/037bf010-d9fb-4db9-9927-6079b8b745cf"
 					(page "14")
 				)

Commit message: Label PEX8780-AB80BI G as the only switch CANDIDATE (DNP).
Keepout is one 35 mm 1156-FCBGA for 8x x8 Gen3 plus one x16 host uplink.
Do not invent a second MPN. Do not stuff. 8-layer is likely if this BGA
is ever assembled; PCBWay 1156-FCBGA attach remains Unknown.

Still do not fabricate or energize P48V. No xGMI, no CEM.

Co-authored-by: zivzancoeli-commits <zivzancoeli-commits@users.noreply.github.com>
Other:
- removed sheet 11_PM8536_DNP
- added sheet 11_PEX8780_CANDIDATE (sheets/11_pcie_switch_unknown.kicad_sch)
- note added: "DO NOT FABRICATE / DO NOT ENERGIZE P48V 8 electrically designed OAM seats (first stuffing: 2 modules / 6 DNP OK — no respin). 16x Molex 218910-1115, 5.00 mm stack. Outline 492 x 372 mm. Generated 12L 2.0 mm. 4x2 of 103x166 mm KOZ = 412x332 mm INFERRED tiling (not a UBB drawing). All 8: named PE toward PEX8780-AB80BI G CANDIDATE DNP (8x x8 + one x16 uplink). No second switch MPN. Host stub: X11DPH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"
- note removed: "DO NOT FABRICATE / DO NOT ENERGIZE P48V 8 electrically designed OAM seats (first stuffing: 2 modules / 6 DNP OK — no respin). 16x Molex 218910-1115, 5.00 mm stack. 12-layer 2.0 mm stuffed-switch TARGET. Outline 492 x 372 mm. 4x2 of 103x166 mm KOZ = 412x332 mm INFERRED tiling (not a UBB drawing). All 8: named PE toward 2x PM8536B-FEI DNP (x8/GCD; SW0=0-3, SW1=4-7). No CEM invented. Host stub: X11D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"
Changed lines of the file:
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@@
         (comment 4 "r2.0 UNUSABLE. P3V3=Conn0 C1/C2. 12L 2.0mm stuffed-switch TARGET. Star-fed P48V.")
 	)
-	(text "DO NOT FABRICATE / DO NOT ENERGIZE P48V\n8 electrically designed OAM seats (first stuffing: 2 modules / 6 DNP OK — no respin).\n16x Molex 218910-1115, 5.00 mm stack. 12-layer 2.0 mm stuffed-switch TARGET. Outline 492 x 372 mm.\n4x2 of 103x166 mm KOZ = 412x332 mm INFERRED tiling (not a UBB drawing).\nAll 8: named PE toward 2x PM8536B-FEI DNP (x8/GCD; SW0=0-3, SW1=4-7). No CEM invented.\nHost stub: X11DPH-T 3x Gen3 x16 + 4x Gen3 x8 keepout. Two CPU x16 = switch uplinks.\nX11DPH-T / NH-D9 DX-3647 / B550M are NOT on this PCB. Chamber A mATX is not this PCB.\nS1-S7 NOT routed (no xGMI). TEST*/RFU/DO_NOT_USE unmapped. PVREF never driven.\nP48V: SB175 long-edge entry + ~15A fuse/seat + LOCAL pours on 16 Conn0 pads. NOT a 100A flood.\nMolex 2026-08-18: CSA 60V (COFC 80170713) at OCP P48V; skip pins = published map, no extra NC.\nOPEN: 1.2 A/contact at 48-59.5 V (2 oz). HOST_PWRGD is ENABLE. No GPU VRM. P12V2 Unknown/may be NC.\nDell D3000E-S1 is 12 V CRPS — do not mix into P48V. P3V3 = Conn0 C1/C2 only. Never r2.0."
+	(text "DO NOT FABRICATE / DO NOT ENERGIZE P48V\n8 electrically designed OAM seats (first stuffing: 2 modules / 6 DNP OK — no respin).\n16x Molex 218910-1115, 5.00 mm stack. Outline 492 x 372 mm. Generated 12L 2.0 mm.\n4x2 of 103x166 mm KOZ = 412x332 mm INFERRED tiling (not a UBB drawing).\nAll 8: named PE toward PEX8780-AB80BI G CANDIDATE DNP (8x x8 + one x16 uplink). No second switch MPN.\nHost stub: X11DPH-T 3x Gen3 x16 + 4x Gen3 x8 keepout. One CPU x16 = switch uplink. No CEM invented.\nX11DPH-T / NH-D9 DX-3647 / B550M are NOT on this PCB. Chamber A mATX is not this PCB.\nS1-S7 NOT routed (no xGMI). TEST*/RFU/DO_NOT_USE unmapped. PVREF never driven.\nP48V: SB175 long-edge entry + ~15A fuse/seat + LOCAL pours on 16 Conn0 pads. NOT a 100A flood.\nMolex 2026-08-18: CSA 60V (COFC 80170713) at OCP P48V; skip pins = published map, no extra NC.\nOPEN: 1.2 A/contact at 48-59.5 V (2 oz). HOST_PWRGD is ENABLE. No GPU VRM. P12V2 Unknown/may be NC.\nDell D3000E-S1 is 12 V CRPS — do not mix into P48V. P3V3 = Conn0 C1/C2 only. Never r2.0."
 		(exclude_from_sim no)
 		(at 25.4 15.24 0)
@@
 		(instances
 			(project "MI250X_8OAM_PCBWay_Chassis_Stub"
-				(path "/037bf010-d9fb-4db9-9927-6079b8b745cf"
+				(path "/e90c8d21-a269-43dd-bc6c-6fbff61026d3"
 					(page "2")
 				)
@@
 		(instances
 			(project "MI250X_8OAM_PCBWay_Chassis_Stub"
-				(path "/037bf010-d9fb-4db9-9927-6079b8b745cf"
+				(path "/e90c8d21-a269-43dd-bc6c-6fbff61026d3"
 					(page "3")
 				)
@@
 		(instances
 			(project "MI250X_8OAM_PCBWay_Chassis_Stub"
-				(path "/037bf010-d9fb-4db9-9927-6079b8b745cf"
+				(path "/e90c8d21-a269-43dd-bc6c-6fbff61026d3"
 					(page "4")
 				)
@@
 		(instances
 			(project "MI250X_8OAM_PCBWay_Chassis_Stub"
-				(path "/037bf010-d9fb-4db9-9927-6079b8b745cf"
+				(path "/e90c8d21-a269-43dd-bc6c-6fbff61026d3"
 					(page "5")
 				)
@@
 		(instances
 			(project "MI250X_8OAM_PCBWay_Chassis_Stub"
-				(path "/037bf010-d9fb-4db9-9927-6079b8b745cf"
+				(path "/e90c8d21-a269-43dd-bc6c-6fbff61026d3"
 					(page "6")
 				)
@@
 		(instances
 			(project "MI250X_8OAM_PCBWay_Chassis_Stub"
-				(path "/037bf010-d9fb-4db9-9927-6079b8b745cf"
+				(path "/e90c8d21-a269-43dd-bc6c-6fbff61026d3"
 					(page "7")
 				)
@@
 		(instances
 			(project "MI250X_8OAM_PCBWay_Chassis_Stub"
-				(path "/037bf010-d9fb-4db9-9927-6079b8b745cf"
+				(path "/e90c8d21-a269-43dd-bc6c-6fbff61026d3"
 					(page "8")
 				)
@@
 		(instances
 			(project "MI250X_8OAM_PCBWay_Chassis_Stub"
-				(path "/037bf010-d9fb-4db9-9927-6079b8b745cf"
+				(path "/e90c8d21-a269-43dd-bc6c-6fbff61026d3"
 					(page "9")
 				)
@@
 		(instances
 			(project "MI250X_8OAM_PCBWay_Chassis_Stub"
-				(path "/037bf010-d9fb-4db9-9927-6079b8b745cf"
+				(path "/e90c8d21-a269-43dd-bc6c-6fbff61026d3"
 					(page "10")
 				)
@@
 		(instances
 			(project "MI250X_8OAM_PCBWay_Chassis_Stub"
-				(path "/037bf010-d9fb-4db9-9927-6079b8b745cf"
+				(path "/e90c8d21-a269-43dd-bc6c-6fbff61026d3"
 					(page "11")
 				)
@@
 		(instances
 			(project "MI250X_8OAM_PCBWay_Chassis_Stub"
-				(path "/037bf010-d9fb-4db9-9927-6079b8b745cf"
+				(path "/e90c8d21-a269-43dd-bc6c-6fbff61026d3"
 					(page "12")
 				)
@@
 		(stroke (width 0.1524) (type solid))
 		(fill (color 0 0 0 0.0000))
-		(property "Sheetname" "11_PM8536_DNP"
+		(property "Sheetname" "11_PEX8780_CANDIDATE"
 			(at 238.54 181.46 0)
 			(effects (font (size 1.27 1.27)) (justify left bottom))
@@
 		(instances
 			(project "MI250X_8OAM_PCBWay_Chassis_Stub"
-				(path "/037bf010-d9fb-4db9-9927-6079b8b745cf"
+				(path "/e90c8d21-a269-43dd-bc6c-6fbff61026d3"
 					(page "13")
 				)
@@
 		(instances
 			(project "MI250X_8OAM_PCBWay_Chassis_Stub"
-				(path "/037bf010-d9fb-4db9-9927-6079b8b745cf"
+				(path "/e90c8d21-a269-43dd-bc6c-6fbff61026d3"
 					(page "14")
 				)

Commit message: Make PM8536B-FEI the PRIMARY switch keepout (DNP x2).
Two 37.5 mm 1311-FCBGA courtyards, x8 per GCD (SW0 seats 0-3, SW1 4-7),
two CPU x16 uplinks. PEX8780 stays a cheaper 80-lane alt in docs only.
GCD1 = SERDES_7 remains Inferred. No CEM, no xGMI, do not fabricate.

Co-authored-by: zivzancoeli-commits <zivzancoeli-commits@users.noreply.github.com>
Other:
- removed sheet 11_PEX8780_CANDIDATE
- added sheet 11_PM8536_DNP (sheets/11_pcie_switch_unknown.kicad_sch)
- note added: "DO NOT FABRICATE / DO NOT ENERGIZE P48V 8 electrically designed OAM seats (first stuffing: 2 modules / 6 DNP OK — no respin). 16x Molex 218910-1115, 5.00 mm stack. 12-layer 2.0 mm stuffed-switch TARGET. Outline 492 x 372 mm. 4x2 of 103x166 mm KOZ = 412x332 mm INFERRED tiling (not a UBB drawing). All 8: named PE toward 2x PM8536B-FEI DNP PRIMARY (x8/GCD; SW0=0-3, SW1=4-7). No CEM invented. Host st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"
- note removed: "DO NOT FABRICATE / DO NOT ENERGIZE P48V 8 electrically designed OAM seats (first stuffing: 2 modules / 6 DNP OK — no respin). 16x Molex 218910-1115, 5.00 mm stack. Outline 492 x 372 mm. Generated 12L 2.0 mm. 4x2 of 103x166 mm KOZ = 412x332 mm INFERRED tiling (not a UBB drawing). All 8: named PE toward PEX8780-AB80BI G CANDIDATE DNP (8x x8 + one x16 uplink). No second switch MPN. Host stub: X11DPH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"
Changed lines of the file:
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@@
         (comment 2 "8 OAM seats. Host X11DPH-T is NOT on this PCB. No CEM cable. No 20-layer UBB.")
         (comment 3 "Pin names: OAM Pin map rev 1.0.xlsx — OCP generic, NOT AMD overlay")
-        (comment 4 "r2.0 UNUSABLE. P3V3=Conn0 C1/C2. 12L 2.0mm stuffed-switch TARGET. Star-fed P48V.")
-	)
-	(text "DO NOT FABRICATE / DO NOT ENERGIZE P48V\n8 electrically designed OAM seats (first stuffing: 2 modules / 6 DNP OK — no respin).\n16x Molex 218910-1115, 5.00 mm stack. Outline 492 x 372 mm. Generated 12L 2.0 mm.\n4x2 of 103x166 mm KOZ = 412x332 mm INFERRED tiling (not a UBB drawing).\nAll 8: named PE toward PEX8780-AB80BI G CANDIDATE DNP (8x x8 + one x16 uplink). No second switch MPN.\nHost stub: X11DPH-T 3x Gen3 x16 + 4x Gen3 x8 keepout. One CPU x16 = switch uplink. No CEM invented.\nX11DPH-T / NH-D9 DX-3647 / B550M are NOT on this PCB. Chamber A mATX is not this PCB.\nS1-S7 NOT routed (no xGMI). TEST*/RFU/DO_NOT_USE unmapped. PVREF never driven.\nP48V: SB175 long-edge entry + ~15A fuse/seat + LOCAL pours on 16 Conn0 pads. NOT a 100A flood.\nMolex 2026-08-18: CSA 60V (COFC 80170713) at OCP P48V; skip pins = published map, no extra NC.\nOPEN: 1.2 A/contact at 48-59.5 V (2 oz). HOST_PWRGD is ENABLE. No GPU VRM. P12V2 Unknown/may be NC.\nDell D3000E-S1 is 12 V CRPS — do not mix into P48V. P3V3 = Conn0 C1/C2 only. Never r2.0."
+        (comment 4 "r2.0 UNUSABLE. P3V3=Conn0 C1/C2. 12L 2.0mm stuffed-switch TARGET. 2x PM8536 DNP. Star-fed P48V.")
+	)
+	(text "DO NOT FABRICATE / DO NOT ENERGIZE P48V\n8 electrically designed OAM seats (first stuffing: 2 modules / 6 DNP OK — no respin).\n16x Molex 218910-1115, 5.00 mm stack. 12-layer 2.0 mm stuffed-switch TARGET. Outline 492 x 372 mm.\n4x2 of 103x166 mm KOZ = 412x332 mm INFERRED tiling (not a UBB drawing).\nAll 8: named PE toward 2x PM8536B-FEI DNP PRIMARY (x8/GCD; SW0=0-3, SW1=4-7). No CEM invented.\nHost stub: X11DPH-T 3x Gen3 x16 + 4x Gen3 x8 keepout. Two CPU x16 = switch uplinks.\nX11DPH-T / NH-D9 DX-3647 / B550M are NOT on this PCB. Chamber A mATX is not this PCB.\nS1-S7 NOT routed (no xGMI). TEST*/RFU/DO_NOT_USE unmapped. PVREF never driven.\nP48V: SB175 long-edge entry + ~15A fuse/seat + LOCAL pours on 16 Conn0 pads. NOT a 100A flood.\nMolex 2026-08-18: CSA 60V (COFC 80170713) at OCP P48V; skip pins = published map, no extra NC.\nOPEN: 1.2 A/contact at 48-59.5 V (2 oz). HOST_PWRGD is ENABLE. No GPU VRM. P12V2 Unknown/may be NC.\nDell D3000E-S1 is 12 V CRPS — do not mix into P48V. P3V3 = Conn0 C1/C2 only. Never r2.0."
 		(exclude_from_sim no)
 		(at 25.4 15.24 0)
@@
 		(instances
 			(project "MI250X_8OAM_PCBWay_Chassis_Stub"
-				(path "/e90c8d21-a269-43dd-bc6c-6fbff61026d3"
+				(path "/d119bf48-350e-4c21-b608-fdd9aec6ebb4"
 					(page "2")
 				)
@@
 		(instances
 			(project "MI250X_8OAM_PCBWay_Chassis_Stub"
-				(path "/e90c8d21-a269-43dd-bc6c-6fbff61026d3"
+				(path "/d119bf48-350e-4c21-b608-fdd9aec6ebb4"
 					(page "3")
 				)
@@
 		(instances
 			(project "MI250X_8OAM_PCBWay_Chassis_Stub"
-				(path "/e90c8d21-a269-43dd-bc6c-6fbff61026d3"
+				(path "/d119bf48-350e-4c21-b608-fdd9aec6ebb4"
 					(page "4")
 				)
@@
 		(instances
 			(project "MI250X_8OAM_PCBWay_Chassis_Stub"
-				(path "/e90c8d21-a269-43dd-bc6c-6fbff61026d3"
+				(path "/d119bf48-350e-4c21-b608-fdd9aec6ebb4"
 					(page "5")
 				)
@@
 		(instances
 			(project "MI250X_8OAM_PCBWay_Chassis_Stub"
-				(path "/e90c8d21-a269-43dd-bc6c-6fbff61026d3"
+				(path "/d119bf48-350e-4c21-b608-fdd9aec6ebb4"
 					(page "6")
 				)
@@
 		(instances
 			(project "MI250X_8OAM_PCBWay_Chassis_Stub"
-				(path "/e90c8d21-a269-43dd-bc6c-6fbff61026d3"
+				(path "/d119bf48-350e-4c21-b608-fdd9aec6ebb4"
 					(page "7")
 				)
@@
 		(instances
 			(project "MI250X_8OAM_PCBWay_Chassis_Stub"
-				(path "/e90c8d21-a269-43dd-bc6c-6fbff61026d3"
+				(path "/d119bf48-350e-4c21-b608-fdd9aec6ebb4"
 					(page "8")
 				)
@@
 		(instances
 			(project "MI250X_8OAM_PCBWay_Chassis_Stub"
-				(path "/e90c8d21-a269-43dd-bc6c-6fbff61026d3"
+				(path "/d119bf48-350e-4c21-b608-fdd9aec6ebb4"
 					(page "9")
 				)
@@
 		(instances
 			(project "MI250X_8OAM_PCBWay_Chassis_Stub"
-				(path "/e90c8d21-a269-43dd-bc6c-6fbff61026d3"
+				(path "/d119bf48-350e-4c21-b608-fdd9aec6ebb4"
 					(page "10")
 				)
@@
 		(instances
 			(project "MI250X_8OAM_PCBWay_Chassis_Stub"
-				(path "/e90c8d21-a269-43dd-bc6c-6fbff61026d3"
+				(path "/d119bf48-350e-4c21-b608-fdd9aec6ebb4"
 					(page "11")
 				)
@@
 		(instances
 			(project "MI250X_8OAM_PCBWay_Chassis_Stub"
-				(path "/e90c8d21-a269-43dd-bc6c-6fbff61026d3"
+				(path "/d119bf48-350e-4c21-b608-fdd9aec6ebb4"
 					(page "12")
 				)
@@
 		(stroke (width 0.1524) (type solid))
 		(fill (color 0 0 0 0.0000))
-		(property "Sheetname" "11_PEX8780_CANDIDATE"
+		(property "Sheetname" "11_PM8536_DNP"
 			(at 238.54 181.46 0)
 			(effects (font (size 1.27 1.27)) (justify left bottom))
@@
 		(instances
 			(project "MI250X_8OAM_PCBWay_Chassis_Stub"
-				(path "/e90c8d21-a269-43dd-bc6c-6fbff61026d3"
+				(path "/d119bf48-350e-4c21-b608-fdd9aec6ebb4"
 					(page "13")
 				)
@@
 		(instances
 			(project "MI250X_8OAM_PCBWay_Chassis_Stub"
-				(path "/e90c8d21-a269-43dd-bc6c-6fbff61026d3"
+				(path "/d119bf48-350e-4c21-b608-fdd9aec6ebb4"
 					(page "14")
 				)
