File: Generated_Project/Rev3_8Seat_PCBWay_Chassis_v1/MI250X_8OAM_PCBWay_Chassis_Stub.kicad_sch (KiCad schematic)
At the start: 0 parts

Commit message: Regenerate 8-seat named-net chassis: all seats electrically designed.
Sheet names seats 2-7 are connectors, not MechPower. Silk/title say named-net
chassis. KiCad 9.0.9 ERC/DRC and top preview refreshed. Do not fabricate,
do not energize P48V, do not upload to PCBWay.

Co-authored-by: zivzancoeli-commits <zivzancoeli-commits@users.noreply.github.com>
Other:
- removed sheet 02_Host_PCIe_Stub_OAM0_1
- removed sheet 05_OAM2_MechPower
- removed sheet 06_OAM3_MechPower
- removed sheet 07_OAM4_MechPower
- removed sheet 08_OAM5_MechPower
- removed sheet 09_OAM6_MechPower
- removed sheet 10_OAM7_MechPower
- added sheet 02_Host_PCIe_Named_8Seat (sheets/02_host_pcie_stub.kicad_sch)
- added sheet 05_OAM2_Connectors (sheets/05_oam2_connectors.kicad_sch)
- added sheet 06_OAM3_Connectors (sheets/06_oam3_connectors.kicad_sch)
- added sheet 07_OAM4_Connectors (sheets/07_oam4_connectors.kicad_sch)
- added sheet 08_OAM5_Connectors (sheets/08_oam5_connectors.kicad_sch)
- added sheet 09_OAM6_Connectors (sheets/09_oam6_connectors.kicad_sch)
- added sheet 10_OAM7_Connectors (sheets/10_oam7_connectors.kicad_sch)
- title: Rev3 8-seat PCBWay chassis stub (NOT fab-ready) -> Rev3 8-seat PCBWay named-net chassis (NOT fab-ready)
Changed lines of the file:
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@@
 	(paper "A3")
 	(title_block
-		(title "Rev3 8-seat PCBWay chassis stub (NOT fab-ready)")
-		(date "2026-08-21")
+		(title "Rev3 8-seat PCBWay named-net chassis (NOT fab-ready)")
+		(date "2026-08-22")
 		(rev "Rev3_8Seat_PCBWay_v1")
         (comment 1 "DO NOT FABRICATE. DO NOT ENERGIZE P48V. Molex 60V written 2026-08-18; 1.2A/contact OPEN.")
@@
 		(instances
 			(project "MI250X_8OAM_PCBWay_Chassis_Stub"
-				(path "/d119bf48-350e-4c21-b608-fdd9aec6ebb4"
+				(path "/300a9d23-e474-4abf-8513-cefb6e5ee91c"
 					(page "2")
 				)
@@
 		(instances
 			(project "MI250X_8OAM_PCBWay_Chassis_Stub"
-				(path "/d119bf48-350e-4c21-b608-fdd9aec6ebb4"
+				(path "/300a9d23-e474-4abf-8513-cefb6e5ee91c"
 					(page "3")
 				)
@@
 		(stroke (width 0.1524) (type solid))
 		(fill (color 0 0 0 0.0000))
-		(property "Sheetname" "02_Host_PCIe_Stub_OAM0_1"
+		(property "Sheetname" "02_Host_PCIe_Named_8Seat"
 			(at 166.54 97.46 0)
 			(effects (font (size 1.27 1.27)) (justify left bottom))
@@
 		(instances
 			(project "MI250X_8OAM_PCBWay_Chassis_Stub"
-				(path "/d119bf48-350e-4c21-b608-fdd9aec6ebb4"
+				(path "/300a9d23-e474-4abf-8513-cefb6e5ee91c"
 					(page "4")
 				)
@@
 		(instances
 			(project "MI250X_8OAM_PCBWay_Chassis_Stub"
-				(path "/d119bf48-350e-4c21-b608-fdd9aec6ebb4"
+				(path "/300a9d23-e474-4abf-8513-cefb6e5ee91c"
 					(page "5")
 				)
@@
 		(instances
 			(project "MI250X_8OAM_PCBWay_Chassis_Stub"
-				(path "/d119bf48-350e-4c21-b608-fdd9aec6ebb4"
+				(path "/300a9d23-e474-4abf-8513-cefb6e5ee91c"
 					(page "6")
 				)
@@
 		(stroke (width 0.1524) (type solid))
 		(fill (color 0 0 0 0.0000))
-		(property "Sheetname" "05_OAM2_MechPower"
+		(property "Sheetname" "05_OAM2_Connectors"
 			(at 94.54 139.46 0)
 			(effects (font (size 1.27 1.27)) (justify left bottom))
@@
 		(instances
 			(project "MI250X_8OAM_PCBWay_Chassis_Stub"
-				(path "/d119bf48-350e-4c21-b608-fdd9aec6ebb4"
+				(path "/300a9d23-e474-4abf-8513-cefb6e5ee91c"
 					(page "7")
 				)
@@
 		(stroke (width 0.1524) (type solid))
 		(fill (color 0 0 0 0.0000))
-		(property "Sheetname" "06_OAM3_MechPower"
+		(property "Sheetname" "06_OAM3_Connectors"
 			(at 166.54 139.46 0)
 			(effects (font (size 1.27 1.27)) (justify left bottom))
@@
 		(instances
 			(project "MI250X_8OAM_PCBWay_Chassis_Stub"
-				(path "/d119bf48-350e-4c21-b608-fdd9aec6ebb4"
+				(path "/300a9d23-e474-4abf-8513-cefb6e5ee91c"
 					(page "8")
 				)
@@
 		(stroke (width 0.1524) (type solid))
 		(fill (color 0 0 0 0.0000))
-		(property "Sheetname" "07_OAM4_MechPower"
+		(property "Sheetname" "07_OAM4_Connectors"
 			(at 238.54 139.46 0)
 			(effects (font (size 1.27 1.27)) (justify left bottom))
@@
 		(instances
 			(project "MI250X_8OAM_PCBWay_Chassis_Stub"
-				(path "/d119bf48-350e-4c21-b608-fdd9aec6ebb4"
+				(path "/300a9d23-e474-4abf-8513-cefb6e5ee91c"
 					(page "9")
 				)
@@
 		(stroke (width 0.1524) (type solid))
 		(fill (color 0 0 0 0.0000))
-		(property "Sheetname" "08_OAM5_MechPower"
+		(property "Sheetname" "08_OAM5_Connectors"
 			(at 22.54 181.46 0)
 			(effects (font (size 1.27 1.27)) (justify left bottom))
@@
 		(instances
 			(project "MI250X_8OAM_PCBWay_Chassis_Stub"
-				(path "/d119bf48-350e-4c21-b608-fdd9aec6ebb4"
+				(path "/300a9d23-e474-4abf-8513-cefb6e5ee91c"
 					(page "10")
 				)
@@
 		(stroke (width 0.1524) (type solid))
 		(fill (color 0 0 0 0.0000))
-		(property "Sheetname" "09_OAM6_MechPower"
+		(property "Sheetname" "09_OAM6_Connectors"
 			(at 94.54 181.46 0)
 			(effects (font (size 1.27 1.27)) (justify left bottom))
@@
 		(instances
 			(project "MI250X_8OAM_PCBWay_Chassis_Stub"
-				(path "/d119bf48-350e-4c21-b608-fdd9aec6ebb4"
+				(path "/300a9d23-e474-4abf-8513-cefb6e5ee91c"
 					(page "11")
 				)
@@
 		(stroke (width 0.1524) (type solid))
 		(fill (color 0 0 0 0.0000))
-		(property "Sheetname" "10_OAM7_MechPower"
+		(property "Sheetname" "10_OAM7_Connectors"
 			(at 166.54 181.46 0)
 			(effects (font (size 1.27 1.27)) (justify left bottom))
@@
 		(instances
 			(project "MI250X_8OAM_PCBWay_Chassis_Stub"
-				(path "/d119bf48-350e-4c21-b608-fdd9aec6ebb4"
+				(path "/300a9d23-e474-4abf-8513-cefb6e5ee91c"
 					(page "12")
 				)
@@
 		(instances
 			(project "MI250X_8OAM_PCBWay_Chassis_Stub"
-				(path "/d119bf48-350e-4c21-b608-fdd9aec6ebb4"
+				(path "/300a9d23-e474-4abf-8513-cefb6e5ee91c"
 					(page "13")
 				)
@@
 		(instances
 			(project "MI250X_8OAM_PCBWay_Chassis_Stub"
-				(path "/d119bf48-350e-4c21-b608-fdd9aec6ebb4"
+				(path "/300a9d23-e474-4abf-8513-cefb6e5ee91c"
 					(page "14")
 				)

Commit message: Add PCBWay-submittable POWER+MECH fab package for the Rev3 8-seat chassis.
Star-fed P48V (SB175 6325G1 + 2x 1382, per-seat 0476015.MR, local Conn0 pours),
THL 40-4812WI and OKI-78SR bucks, filled 12L 2.0 mm Gerbers/drill/IPC-356/PnP.
PM8536 stays DNP. Silk keeps DO NOT ENERGIZE P48V. Do not upload from this agent.

Co-authored-by: zivzancoeli-commits <zivzancoeli-commits@users.noreply.github.com>
Other:
- note added: "DO NOT ENERGIZE P48V — POWER+MECH first article (PM8536 DNP) 8 electrically designed OAM seats (first stuffing: 2 modules / 6 DNP OK — no respin). 16x Molex 218910-1115, 5.00 mm stack. 12-layer 2.0 mm stuffed-switch TARGET. Outline 492 x 372 mm. 4x2 of 103x166 mm KOZ = 412x332 mm INFERRED tiling (not a UBB drawing). All 8: named PE toward 2x PM8536B-FEI DNP PRIMARY (x8/GCD; SW0=0-3, SW1=4-7). No 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"
- note removed: "DO NOT FABRICATE / DO NOT ENERGIZE P48V 8 electrically designed OAM seats (first stuffing: 2 modules / 6 DNP OK — no respin). 16x Molex 218910-1115, 5.00 mm stack. 12-layer 2.0 mm stuffed-switch TARGET. Outline 492 x 372 mm. 4x2 of 103x166 mm KOZ = 412x332 mm INFERRED tiling (not a UBB drawing). All 8: named PE toward 2x PM8536B-FEI DNP PRIMARY (x8/GCD; SW0=0-3, SW1=4-7). No CEM invented. Host st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"
- title: Rev3 8-seat PCBWay named-net chassis (NOT fab-ready) -> Rev3 8-seat PCBWay POWER+MECH first article (DO NOT ENERGIZE P48V)
Changed lines of the file:
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@@
 	(paper "A3")
 	(title_block
-		(title "Rev3 8-seat PCBWay named-net chassis (NOT fab-ready)")
+		(title "Rev3 8-seat PCBWay POWER+MECH first article (DO NOT ENERGIZE P48V)")
 		(date "2026-08-22")
 		(rev "Rev3_8Seat_PCBWay_v1")
-        (comment 1 "DO NOT FABRICATE. DO NOT ENERGIZE P48V. Molex 60V written 2026-08-18; 1.2A/contact OPEN.")
+        (comment 1 "DO NOT ENERGIZE P48V. Molex 60V written 2026-08-18; 1.2A/contact OPEN. Skip-pin NC.")
         (comment 2 "8 OAM seats. Host X11DPH-T is NOT on this PCB. No CEM cable. No 20-layer UBB.")
         (comment 3 "Pin names: OAM Pin map rev 1.0.xlsx — OCP generic, NOT AMD overlay")
         (comment 4 "r2.0 UNUSABLE. P3V3=Conn0 C1/C2. 12L 2.0mm stuffed-switch TARGET. 2x PM8536 DNP. Star-fed P48V.")
 	)
-	(text "DO NOT FABRICATE / DO NOT ENERGIZE P48V\n8 electrically designed OAM seats (first stuffing: 2 modules / 6 DNP OK — no respin).\n16x Molex 218910-1115, 5.00 mm stack. 12-layer 2.0 mm stuffed-switch TARGET. Outline 492 x 372 mm.\n4x2 of 103x166 mm KOZ = 412x332 mm INFERRED tiling (not a UBB drawing).\nAll 8: named PE toward 2x PM8536B-FEI DNP PRIMARY (x8/GCD; SW0=0-3, SW1=4-7). No CEM invented.\nHost stub: X11DPH-T 3x Gen3 x16 + 4x Gen3 x8 keepout. Two CPU x16 = switch uplinks.\nX11DPH-T / NH-D9 DX-3647 / B550M are NOT on this PCB. Chamber A mATX is not this PCB.\nS1-S7 NOT routed (no xGMI). TEST*/RFU/DO_NOT_USE unmapped. PVREF never driven.\nP48V: SB175 long-edge entry + ~15A fuse/seat + LOCAL pours on 16 Conn0 pads. NOT a 100A flood.\nMolex 2026-08-18: CSA 60V (COFC 80170713) at OCP P48V; skip pins = published map, no extra NC.\nOPEN: 1.2 A/contact at 48-59.5 V (2 oz). HOST_PWRGD is ENABLE. No GPU VRM. P12V2 Unknown/may be NC.\nDell D3000E-S1 is 12 V CRPS — do not mix into P48V. P3V3 = Conn0 C1/C2 only. Never r2.0."
+	(text "DO NOT ENERGIZE P48V — POWER+MECH first article (PM8536 DNP)\n8 electrically designed OAM seats (first stuffing: 2 modules / 6 DNP OK — no respin).\n16x Molex 218910-1115, 5.00 mm stack. 12-layer 2.0 mm stuffed-switch TARGET. Outline 492 x 372 mm.\n4x2 of 103x166 mm KOZ = 412x332 mm INFERRED tiling (not a UBB drawing).\nAll 8: named PE toward 2x PM8536B-FEI DNP PRIMARY (x8/GCD; SW0=0-3, SW1=4-7). No CEM invented.\nHost stub: X11DPH-T 3x Gen3 x16 + 4x Gen3 x8 keepout. Two CPU x16 = switch uplinks.\nX11DPH-T / NH-D9 DX-3647 / B550M are NOT on this PCB. Chamber A mATX is not this PCB.\nS1-S7 NOT routed (no xGMI). TEST*/RFU/DO_NOT_USE unmapped. PVREF never driven.\nP48V: SB175 (6325G1+2x1382) + 0476015.MR 15A/seat + LOCAL pours. NOT a 100A flood.\nMolex 2026-08-18: CSA 60V (COFC 80170713) at OCP P48V; skip pins = published map, no extra NC.\nOPEN: 1.2 A/contact at 48-59.5 V (2 oz). HOST_PWRGD is ENABLE. No GPU VRM. P12V2 Unknown/may be NC.\nDell D3000E-S1 is 12 V CRPS — do not mix into P48V. P3V3 = Conn0 C1/C2 only. Never r2.0."
 		(exclude_from_sim no)
 		(at 25.4 15.24 0)
@@
 		(instances
 			(project "MI250X_8OAM_PCBWay_Chassis_Stub"
-				(path "/300a9d23-e474-4abf-8513-cefb6e5ee91c"
+				(path "/828fc2f0-8739-4d6c-8db1-826eb1db204f"
 					(page "2")
 				)
@@
 		(instances
 			(project "MI250X_8OAM_PCBWay_Chassis_Stub"
-				(path "/300a9d23-e474-4abf-8513-cefb6e5ee91c"
+				(path "/828fc2f0-8739-4d6c-8db1-826eb1db204f"
 					(page "3")
 				)
@@
 		(instances
 			(project "MI250X_8OAM_PCBWay_Chassis_Stub"
-				(path "/300a9d23-e474-4abf-8513-cefb6e5ee91c"
+				(path "/828fc2f0-8739-4d6c-8db1-826eb1db204f"
 					(page "4")
 				)
@@
 		(instances
 			(project "MI250X_8OAM_PCBWay_Chassis_Stub"
-				(path "/300a9d23-e474-4abf-8513-cefb6e5ee91c"
+				(path "/828fc2f0-8739-4d6c-8db1-826eb1db204f"
 					(page "5")
 				)
@@
 		(instances
 			(project "MI250X_8OAM_PCBWay_Chassis_Stub"
-				(path "/300a9d23-e474-4abf-8513-cefb6e5ee91c"
+				(path "/828fc2f0-8739-4d6c-8db1-826eb1db204f"
 					(page "6")
 				)
@@
 		(instances
 			(project "MI250X_8OAM_PCBWay_Chassis_Stub"
-				(path "/300a9d23-e474-4abf-8513-cefb6e5ee91c"
+				(path "/828fc2f0-8739-4d6c-8db1-826eb1db204f"
 					(page "7")
 				)
@@
 		(instances
 			(project "MI250X_8OAM_PCBWay_Chassis_Stub"
-				(path "/300a9d23-e474-4abf-8513-cefb6e5ee91c"
+				(path "/828fc2f0-8739-4d6c-8db1-826eb1db204f"
 					(page "8")
 				)
@@
 		(instances
 			(project "MI250X_8OAM_PCBWay_Chassis_Stub"
-				(path "/300a9d23-e474-4abf-8513-cefb6e5ee91c"
+				(path "/828fc2f0-8739-4d6c-8db1-826eb1db204f"
 					(page "9")
 				)
@@
 		(instances
 			(project "MI250X_8OAM_PCBWay_Chassis_Stub"
-				(path "/300a9d23-e474-4abf-8513-cefb6e5ee91c"
+				(path "/828fc2f0-8739-4d6c-8db1-826eb1db204f"
 					(page "10")
 				)
@@
 		(instances
 			(project "MI250X_8OAM_PCBWay_Chassis_Stub"
-				(path "/300a9d23-e474-4abf-8513-cefb6e5ee91c"
+				(path "/828fc2f0-8739-4d6c-8db1-826eb1db204f"
 					(page "11")
 				)
@@
 		(instances
 			(project "MI250X_8OAM_PCBWay_Chassis_Stub"
-				(path "/300a9d23-e474-4abf-8513-cefb6e5ee91c"
+				(path "/828fc2f0-8739-4d6c-8db1-826eb1db204f"
 					(page "12")
 				)
@@
 		(instances
 			(project "MI250X_8OAM_PCBWay_Chassis_Stub"
-				(path "/300a9d23-e474-4abf-8513-cefb6e5ee91c"
+				(path "/828fc2f0-8739-4d6c-8db1-826eb1db204f"
 					(page "13")
 				)
@@
 		(instances
 			(project "MI250X_8OAM_PCBWay_Chassis_Stub"
-				(path "/300a9d23-e474-4abf-8513-cefb6e5ee91c"
+				(path "/828fc2f0-8739-4d6c-8db1-826eb1db204f"
 					(page "14")
 				)

Commit message: Make the Rev3 8-seat chassis full-width capable with four PM8536 DNP courtyards.
Same 492x372 POWER+MECH PCB; architecture is now 16 named x16 PE buses
(PE_Sn_GCD0_x16 + PE_Sn_GCD1_x16) and SW0-SW3 keepouts. Two 96-lane
switches are enough for 8x x8/GCD, not 8x x16/GCD. Host stays X11DPH-T
(~80 lanes) and cannot light 256 downstream. Do not energize P48V.

Co-authored-by: zivzancoeli-commits <zivzancoeli-commits@users.noreply.github.com>
Other:
- removed sheet 11_PM8536_DNP
- added sheet 11_PM8536_DNP_x4 (sheets/11_pcie_switch_unknown.kicad_sch)
- note added: "DO NOT ENERGIZE P48V — POWER+MECH first article (4x PM8536 DNP) 8 electrically designed OAM seats. Populate 2 (0-1) then 4 (0-3) then 8 — no respin. 16x Molex 218910-1115, 5.00 mm stack. 12-layer 2.0 mm stuffed-switch TARGET. Outline 492 x 372 mm. 4x2 of 103x166 mm KOZ = 412x332 mm INFERRED tiling (not a UBB drawing). FULL-WIDTH CAPABLE: 16x x16 PE names (PE_Sn_GCD0_x16 + PE_Sn_GCD1_x16) toward 4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"
- note removed: "DO NOT ENERGIZE P48V — POWER+MECH first article (PM8536 DNP) 8 electrically designed OAM seats (first stuffing: 2 modules / 6 DNP OK — no respin). 16x Molex 218910-1115, 5.00 mm stack. 12-layer 2.0 mm stuffed-switch TARGET. Outline 492 x 372 mm. 4x2 of 103x166 mm KOZ = 412x332 mm INFERRED tiling (not a UBB drawing). All 8: named PE toward 2x PM8536B-FEI DNP PRIMARY (x8/GCD; SW0=0-3, SW1=4-7). No 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"
Changed lines of the file:
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@@
 		(rev "Rev3_8Seat_PCBWay_v1")
         (comment 1 "DO NOT ENERGIZE P48V. Molex 60V written 2026-08-18; 1.2A/contact OPEN. Skip-pin NC.")
-        (comment 2 "8 OAM seats. Host X11DPH-T is NOT on this PCB. No CEM cable. No 20-layer UBB.")
+        (comment 2 "8 OAM seats. Host X11DPH-T is NOT on this PCB. Chassis full-width capable; host cannot light 256 DS. No CEM cable.")
         (comment 3 "Pin names: OAM Pin map rev 1.0.xlsx — OCP generic, NOT AMD overlay")
-        (comment 4 "r2.0 UNUSABLE. P3V3=Conn0 C1/C2. 12L 2.0mm stuffed-switch TARGET. 2x PM8536 DNP. Star-fed P48V.")
-	)
-	(text "DO NOT ENERGIZE P48V — POWER+MECH first article (PM8536 DNP)\n8 electrically designed OAM seats (first stuffing: 2 modules / 6 DNP OK — no respin).\n16x Molex 218910-1115, 5.00 mm stack. 12-layer 2.0 mm stuffed-switch TARGET. Outline 492 x 372 mm.\n4x2 of 103x166 mm KOZ = 412x332 mm INFERRED tiling (not a UBB drawing).\nAll 8: named PE toward 2x PM8536B-FEI DNP PRIMARY (x8/GCD; SW0=0-3, SW1=4-7). No CEM invented.\nHost stub: X11DPH-T 3x Gen3 x16 + 4x Gen3 x8 keepout. Two CPU x16 = switch uplinks.\nX11DPH-T / NH-D9 DX-3647 / B550M are NOT on this PCB. Chamber A mATX is not this PCB.\nS1-S7 NOT routed (no xGMI). TEST*/RFU/DO_NOT_USE unmapped. PVREF never driven.\nP48V: SB175 (6325G1+2x1382) + 0476015.MR 15A/seat + LOCAL pours. NOT a 100A flood.\nMolex 2026-08-18: CSA 60V (COFC 80170713) at OCP P48V; skip pins = published map, no extra NC.\nOPEN: 1.2 A/contact at 48-59.5 V (2 oz). HOST_PWRGD is ENABLE. No GPU VRM. P12V2 Unknown/may be NC.\nDell D3000E-S1 is 12 V CRPS — do not mix into P48V. P3V3 = Conn0 C1/C2 only. Never r2.0."
+        (comment 4 "r2.0 UNUSABLE. P3V3=Conn0 C1/C2. 12L 2.0mm stuffed-switch TARGET. 4x PM8536 DNP. Star-fed P48V.")
+	)
+	(text "DO NOT ENERGIZE P48V — POWER+MECH first article (4x PM8536 DNP)\n8 electrically designed OAM seats. Populate 2 (0-1) then 4 (0-3) then 8 — no respin.\n16x Molex 218910-1115, 5.00 mm stack. 12-layer 2.0 mm stuffed-switch TARGET. Outline 492 x 372 mm.\n4x2 of 103x166 mm KOZ = 412x332 mm INFERRED tiling (not a UBB drawing).\nFULL-WIDTH CAPABLE: 16x x16 PE names (PE_Sn_GCD0_x16 + PE_Sn_GCD1_x16) toward 4x PM8536B-FEI DNP.\nChassis can SIT/WIRE 8 full-width. Host X11DPH-T ~80 lanes CANNOT LIGHT 256 DS. No CEM invented.\nX11DPH-T / NH-D9 DX-3647 / B550M are NOT on this PCB. Do not swap or design the host board.\nS1-S7 NOT routed (no xGMI). TEST*/RFU/DO_NOT_USE unmapped. PVREF never driven.\nP48V: SB175 (6325G1+2x1382) + 0476015.MR 15A/seat + LOCAL pours. NOT a 100A flood.\nMolex 2026-08-18: CSA 60V (COFC 80170713) at OCP P48V; skip pins = published map, no extra NC.\nOPEN: 1.2 A/contact at 48-59.5 V (2 oz). HOST_PWRGD is ENABLE. No GPU VRM. P12V2 Unknown/may be NC.\nDell D3000E-S1 is 12 V CRPS — do not mix into P48V. P3V3 = Conn0 C1/C2 only. Never r2.0."
 		(exclude_from_sim no)
 		(at 25.4 15.24 0)
@@
 		(instances
 			(project "MI250X_8OAM_PCBWay_Chassis_Stub"
-				(path "/828fc2f0-8739-4d6c-8db1-826eb1db204f"
+				(path "/55d1fb6f-3b8f-4a23-aee7-008dfc99f7b0"
 					(page "2")
 				)
@@
 		(instances
 			(project "MI250X_8OAM_PCBWay_Chassis_Stub"
-				(path "/828fc2f0-8739-4d6c-8db1-826eb1db204f"
+				(path "/55d1fb6f-3b8f-4a23-aee7-008dfc99f7b0"
 					(page "3")
 				)
@@
 		(instances
 			(project "MI250X_8OAM_PCBWay_Chassis_Stub"
-				(path "/828fc2f0-8739-4d6c-8db1-826eb1db204f"
+				(path "/55d1fb6f-3b8f-4a23-aee7-008dfc99f7b0"
 					(page "4")
 				)
@@
 		(instances
 			(project "MI250X_8OAM_PCBWay_Chassis_Stub"
-				(path "/828fc2f0-8739-4d6c-8db1-826eb1db204f"
+				(path "/55d1fb6f-3b8f-4a23-aee7-008dfc99f7b0"
 					(page "5")
 				)
@@
 		(instances
 			(project "MI250X_8OAM_PCBWay_Chassis_Stub"
-				(path "/828fc2f0-8739-4d6c-8db1-826eb1db204f"
+				(path "/55d1fb6f-3b8f-4a23-aee7-008dfc99f7b0"
 					(page "6")
 				)
@@
 		(instances
 			(project "MI250X_8OAM_PCBWay_Chassis_Stub"
-				(path "/828fc2f0-8739-4d6c-8db1-826eb1db204f"
+				(path "/55d1fb6f-3b8f-4a23-aee7-008dfc99f7b0"
 					(page "7")
 				)
@@
 		(instances
 			(project "MI250X_8OAM_PCBWay_Chassis_Stub"
-				(path "/828fc2f0-8739-4d6c-8db1-826eb1db204f"
+				(path "/55d1fb6f-3b8f-4a23-aee7-008dfc99f7b0"
 					(page "8")
 				)
@@
 		(instances
 			(project "MI250X_8OAM_PCBWay_Chassis_Stub"
-				(path "/828fc2f0-8739-4d6c-8db1-826eb1db204f"
+				(path "/55d1fb6f-3b8f-4a23-aee7-008dfc99f7b0"
 					(page "9")
 				)
@@
 		(instances
 			(project "MI250X_8OAM_PCBWay_Chassis_Stub"
-				(path "/828fc2f0-8739-4d6c-8db1-826eb1db204f"
+				(path "/55d1fb6f-3b8f-4a23-aee7-008dfc99f7b0"
 					(page "10")
 				)
@@
 		(instances
 			(project "MI250X_8OAM_PCBWay_Chassis_Stub"
-				(path "/828fc2f0-8739-4d6c-8db1-826eb1db204f"
+				(path "/55d1fb6f-3b8f-4a23-aee7-008dfc99f7b0"
 					(page "11")
 				)
@@
 		(instances
 			(project "MI250X_8OAM_PCBWay_Chassis_Stub"
-				(path "/828fc2f0-8739-4d6c-8db1-826eb1db204f"
+				(path "/55d1fb6f-3b8f-4a23-aee7-008dfc99f7b0"
 					(page "12")
 				)
@@
 		(stroke (width 0.1524) (type solid))
 		(fill (color 0 0 0 0.0000))
-		(property "Sheetname" "11_PM8536_DNP"
+		(property "Sheetname" "11_PM8536_DNP_x4"
 			(at 238.54 181.46 0)
 			(effects (font (size 1.27 1.27)) (justify left bottom))
@@
 		(instances
 			(project "MI250X_8OAM_PCBWay_Chassis_Stub"
-				(path "/828fc2f0-8739-4d6c-8db1-826eb1db204f"
+				(path "/55d1fb6f-3b8f-4a23-aee7-008dfc99f7b0"
 					(page "13")
 				)
@@
 		(instances
 			(project "MI250X_8OAM_PCBWay_Chassis_Stub"
-				(path "/828fc2f0-8739-4d6c-8db1-826eb1db204f"
+				(path "/55d1fb6f-3b8f-4a23-aee7-008dfc99f7b0"
 					(page "14")
 				)
