File: Generated_Project/Rev3_8Seat_PCBWay_Chassis_v1/sheets/02_host_pcie_stub.kicad_sch (KiCad schematic)
At the start: 0 parts

Commit message: Make the Rev3 8-seat chassis full-width capable with four PM8536 DNP courtyards.
Same 492x372 POWER+MECH PCB; architecture is now 16 named x16 PE buses
(PE_Sn_GCD0_x16 + PE_Sn_GCD1_x16) and SW0-SW3 keepouts. Two 96-lane
switches are enough for 8x x8/GCD, not 8x x16/GCD. Host stays X11DPH-T
(~80 lanes) and cannot light 256 downstream. Do not energize P48V.

Co-authored-by: zivzancoeli-commits <zivzancoeli-commits@users.noreply.github.com>
Other:
- note added: "PURPOSE: Named v1.0 PCIE_TXnP/N and PCIE_RXnP/N (n=0..15) on ALL 8 seats plus 16 architectural x16 PE names (full-width capable chassis). 8 electrically designed seats. Populate 2 (seats 0-1) then 4 (0-3) then 8 — the PCB does not require a respin. OCP pin list (module POV): - PETp/n = module TX, host RX. AC caps on motherboard/carrier — not placed. - PERp/n = module RX, host TX. AC caps on mothe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"
- note removed: "PURPOSE: Named v1.0 PCIE_TXnP/N and PCIE_RXnP/N (n=0..15) on ALL 8 seats. 8 electrically designed seats. First stuffing may populate 2 modules / 6 DNP — the PCB does not require a respin for the other six. OCP pin list (module POV): - PETp/n = module TX, host RX. AC caps on motherboard/carrier — not placed. - PERp/n = module RX, host TX. AC caps on motherboard/carrier — not placed. This sheet doe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"
- title: Host PE stub (all 8 seats via DNP PM8536 PRIMARY) -> Host PE stub (16x x16 names, 4x PM8536 DNP)
Changed lines of the file:
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@@
 	(paper "A3")
 	(title_block
-		(title "Host PE stub (all 8 seats via DNP PM8536 PRIMARY)")
+		(title "Host PE stub (16x x16 names, 4x PM8536 DNP)")
 		(date "2026-08-22")
 		(rev "Rev3_8Seat_PCBWay_v1")
@@
         (comment 2 "Documentation sheet — no invented nets")
         (comment 3 "Pin names: OAM Pin map rev 1.0.xlsx — OCP generic, NOT AMD overlay")
-        (comment 4 "r2.0 UNUSABLE. P3V3=Conn0 C1/C2. 12L 2.0mm stuffed-switch TARGET. 2x PM8536 DNP. Star-fed P48V.")
-	)
-	(text "PURPOSE: Named v1.0 PCIE_TXnP/N and PCIE_RXnP/N (n=0..15) on ALL 8 seats.\n\n8 electrically designed seats. First stuffing may populate 2 modules / 6 DNP —\nthe PCB does not require a respin for the other six.\n\nOCP pin list (module POV):\n- PETp/n = module TX, host RX. AC caps on motherboard/carrier — not placed.\n- PERp/n = module RX, host TX. AC caps on motherboard/carrier — not placed.\n\nThis sheet does NOT map those pairs onto a CEM x16 connector pinout.\nDo NOT invent a CEM cable, SlimSAS, MCIO, or retimer BOM.\n\nIntended 8x topology (PRIMARY DNP until stuffed):\n- Two Microchip PM8536B-FEI (Switchtec PFX 96-lane Gen3, 1311-ball 37.5 mm FCBGA, 1.0 mm).\n  ~$460-475, ~18 wk. PCBWay can assemble 1.0 mm without HDI; plan 12-16 layers (not 4).\n  SW0 = seats 0-3 (16 US + 64 DS). SW1 = seats 4-7. x8 per GCD.\n- Each MI250X GCD has its own PCIe Gen4 x16 (AMD + Hot Chips 34). Host trains Gen3.\n- OAM v1.5: one PE x16 on Conn0; a second host x16 may be SERDES_7 on Conn1.\n  GCD1 = SERDES_7 is Inferred — there is NO public AMD overlay proving it.\n  Do not route S1-S7 as if that were proven. No xGMI.\n- Each seat's 16 named PE lanes = 2x x8 (GCD0/GCD1 split is planning; PE_BIF AMD-unknown).\n- Host X11DPH-T (NOT on this PCB): 3x Gen3 x16 + 4x Gen3 x8 = 80 Gen3 lanes.\n  Two CPU x16 = switch uplinks (silk + connector keepout, MPN Unknown).\n  Remaining 1x x16 + 4x x8 unused on this chassis.\n\n8 x 2 x x16 = 256 downstream vs 80 host Gen3 — do not attempt x16-per-GCD.\nPEX8780-AB80BI G (80-lane 35 mm) is a cheaper alt in docs only — not placed.\nPM8533B-F3EI (48-lane 27 mm) is a 2-seat alt in docs only — not placed.\n\nX11DPH-T is NOT a part on this PCB. Chamber A B550M is NOT this PCB.\n"
+        (comment 4 "r2.0 UNUSABLE. P3V3=Conn0 C1/C2. 12L 2.0mm stuffed-switch TARGET. 4x PM8536 DNP. Star-fed P48V.")
+	)
+	(text "PURPOSE: Named v1.0 PCIE_TXnP/N and PCIE_RXnP/N (n=0..15) on ALL 8 seats\nplus 16 architectural x16 PE names (full-width capable chassis).\n\n8 electrically designed seats. Populate 2 (seats 0-1) then 4 (0-3) then 8 —\nthe PCB does not require a respin.\n\nOCP pin list (module POV):\n- PETp/n = module TX, host RX. AC caps on motherboard/carrier — not placed.\n- PERp/n = module RX, host TX. AC caps on motherboard/carrier — not placed.\n\nThis sheet does NOT map those pairs onto a CEM x16 connector pinout.\nDo NOT invent a CEM cable, SlimSAS, MCIO, or retimer BOM.\nDo NOT invent PE pin numbers or assign GCD1 onto S1-S7.\n\nArchitectural names (hierarchical labels; not a fake BGA pinout):\n- PE_S{n}_GCD0_x16 = Conn0 16-lane PCIE bus (OCP-named pads OAM{n}_PCIE_*).\n- PE_S{n}_GCD1_x16 = named only. Overlay Unknown. SERDES_7 as GCD1 PE is Inferred.\n  Pins not assigned. Not S1-S7.\n- PE_SW{k}_US_x16 = four host-facing x16 keepouts toward X11DPH-T.\n\nLane math (verified; not a locked root cause / not a ball map):\n- Full width = 8 modules x 2 GCD x x16 = 256 downstream lanes on the carrier.\n- PM8536B-FEI = 96-lane Gen3, 1311-ball 37.5 mm FCBGA 1.0 mm. Ball map not public.\n- 2x96 = 192. Even with 16 US/switch: 160 DS — enough for 8x x8/GCD (128 DS), NOT 256 DS.\n- 4x96 = 384. Hypothesis partition: each SW 16 US + 64 DS (2 seats x 2 GCD x x16)\n  = 80 of 96, 16 spare. 4 x 16 US = 64 host-facing vs X11DPH-T ~80.\n- Chassis can SIT and be WIRED for 8 full-width. This host CANNOT LIGHT 256 DS.\n  Memory/CPU mix (2x Gold 6230, 64 GB DRAM + 1 TB PMem) does NOT add PCIe lanes.\n- x8/GCD remains a stuffing option if only SW0+SW1 are populated.\n\nSW0 = seats 0-1 (first stuff). SW1 = 2-3. SW2 = 4-5. SW3 = 6-7.\nPEX8780-AB80BI G (80-lane 35 mm) is a cheaper alt in docs only — not placed.\nPM8533B-F3EI (48-lane 27 mm) is a 2-seat alt in docs only — not placed.\n\nX11DPH-T is NOT a part on this PCB. Do not swap or design a host board.\nChamber A B550M is NOT this PCB.\n"
 		(exclude_from_sim no)
 		(at 20.32 20.32 0)
@@
 		(effects (font (size 1.27 1.27)) (justify left))
 	)
+	(hierarchical_label "PE_S0_GCD0_x16"
+		(shape bidirectional)
+		(at 200 130 0)
+		(effects (font (size 1.27 1.27)) (justify left))
+	)
+	(hierarchical_label "PE_S0_GCD1_x16"
+		(shape bidirectional)
+		(at 200 136.0 0)
+		(effects (font (size 1.27 1.27)) (justify left))
+	)
+	(hierarchical_label "PE_S1_GCD0_x16"
+		(shape bidirectional)
+		(at 200 142.0 0)
+		(effects (font (size 1.27 1.27)) (justify left))
+	)
+	(hierarchical_label "PE_S1_GCD1_x16"
+		(shape bidirectional)
+		(at 200 148.0 0)
+		(effects (font (size 1.27 1.27)) (justify left))
+	)
+	(hierarchical_label "PE_S2_GCD0_x16"
+		(shape bidirectional)
+		(at 200 154.0 0)
+		(effects (font (size 1.27 1.27)) (justify left))
+	)
+	(hierarchical_label "PE_S2_GCD1_x16"
+		(shape bidirectional)
+		(at 200 160.0 0)
+		(effects (font (size 1.27 1.27)) (justify left))
+	)
+	(hierarchical_label "PE_S3_GCD0_x16"
+		(shape bidirectional)
+		(at 200 166.0 0)
+		(effects (font (size 1.27 1.27)) (justify left))
+	)
+	(hierarchical_label "PE_S3_GCD1_x16"
+		(shape bidirectional)
+		(at 200 172.0 0)
+		(effects (font (size 1.27 1.27)) (justify left))
+	)
+	(hierarchical_label "PE_S4_GCD0_x16"
+		(shape bidirectional)
+		(at 200 178.0 0)
+		(effects (font (size 1.27 1.27)) (justify left))
+	)
+	(hierarchical_label "PE_S4_GCD1_x16"
+		(shape bidirectional)
+		(at 200 184.0 0)
+		(effects (font (size 1.27 1.27)) (justify left))
+	)
+	(hierarchical_label "PE_S5_GCD0_x16"
+		(shape bidirectional)
+		(at 200 190.0 0)
+		(effects (font (size 1.27 1.27)) (justify left))
+	)
+	(hierarchical_label "PE_S5_GCD1_x16"
+		(shape bidirectional)
+		(at 200 196.0 0)
+		(effects (font (size 1.27 1.27)) (justify left))
+	)
+	(hierarchical_label "PE_S6_GCD0_x16"
+		(shape bidirectional)
+		(at 200 202.0 0)
+		(effects (font (size 1.27 1.27)) (justify left))
+	)
+	(hierarchical_label "PE_S6_GCD1_x16"
+		(shape bidirectional)
+		(at 200 208.0 0)
+		(effects (font (size 1.27 1.27)) (justify left))
+	)
+	(hierarchical_label "PE_S7_GCD0_x16"
+		(shape bidirectional)
+		(at 200 214.0 0)
+		(effects (font (size 1.27 1.27)) (justify left))
+	)
+	(hierarchical_label "PE_S7_GCD1_x16"
+		(shape bidirectional)
+		(at 200 220.0 0)
+		(effects (font (size 1.27 1.27)) (justify left))
+	)
+	(hierarchical_label "PE_SW0_US_x16"
+		(shape bidirectional)
+		(at 200 226.0 0)
+		(effects (font (size 1.27 1.27)) (justify left))
+	)
+	(hierarchical_label "PE_SW1_US_x16"
+		(shape bidirectional)
+		(at 200 232.0 0)
+		(effects (font (size 1.27 1.27)) (justify left))
+	)
+	(hierarchical_label "PE_SW2_US_x16"
+		(shape bidirectional)
+		(at 200 238.0 0)
+		(effects (font (size 1.27 1.27)) (justify left))
+	)
+	(hierarchical_label "PE_SW3_US_x16"
+		(shape bidirectional)
+		(at 200 244.0 0)
+		(effects (font (size 1.27 1.27)) (justify left))
+	)

Commit message: Retarget Rev3 first article to seats 0-1 GCD0 x16 (2-module path).
Same 8-seat PCB. Without overlay, 2x MI250X means two modules can sit
and at most GCD0 on each can be named toward the host keepout (2 GCDs),
not 2x full-width (4 GCDs). Conn0 OCP PCIE_* is the only legal host PE.
No CEM/MCIO MPN. Do not energize P48V.

Co-authored-by: zivzancoeli-commits <zivzancoeli-commits@users.noreply.github.com>
Other:
- note added: "PURPOSE: Named v1.0 PCIE_TXnP/N and PCIE_RXnP/N (n=0..15) on ALL 8 seats. FIRST ARTICLE TARGET: seats 0 and 1. Same 8-seat PCB; 2→4→8 later. Pinmap (Verified OCP v1.0 generic map + pin list; NOT an AMD overlay): - Conn0 PCIE_TX/RX0-15 P/N = 64 pads = PETp/n + PERp/n [15:0] "PCIe or equivalent host link". That is the only legal named host PE today. Call it GCD0 x16 (architectural name). - Conn1 ha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"
- note removed: "PURPOSE: Named v1.0 PCIE_TXnP/N and PCIE_RXnP/N (n=0..15) on ALL 8 seats plus 16 architectural x16 PE names (full-width capable chassis). 8 electrically designed seats. Populate 2 (seats 0-1) then 4 (0-3) then 8 — the PCB does not require a respin. OCP pin list (module POV): - PETp/n = module TX, host RX. AC caps on motherboard/carrier — not placed. - PERp/n = module RX, host TX. AC caps on mothe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"
- title: Host PE stub (16x x16 names, 4x PM8536 DNP) -> Host PE: 2-mod first article GCD0 x16; later-seat names kept
Changed lines of the file:
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@@
 	(paper "A3")
 	(title_block
-		(title "Host PE stub (16x x16 names, 4x PM8536 DNP)")
+		(title "Host PE: 2-mod first article GCD0 x16; later-seat names kept")
 		(date "2026-08-22")
 		(rev "Rev3_8Seat_PCBWay_v1")
@@
         (comment 4 "r2.0 UNUSABLE. P3V3=Conn0 C1/C2. 12L 2.0mm stuffed-switch TARGET. 4x PM8536 DNP. Star-fed P48V.")
 	)
-	(text "PURPOSE: Named v1.0 PCIE_TXnP/N and PCIE_RXnP/N (n=0..15) on ALL 8 seats\nplus 16 architectural x16 PE names (full-width capable chassis).\n\n8 electrically designed seats. Populate 2 (seats 0-1) then 4 (0-3) then 8 —\nthe PCB does not require a respin.\n\nOCP pin list (module POV):\n- PETp/n = module TX, host RX. AC caps on motherboard/carrier — not placed.\n- PERp/n = module RX, host TX. AC caps on motherboard/carrier — not placed.\n\nThis sheet does NOT map those pairs onto a CEM x16 connector pinout.\nDo NOT invent a CEM cable, SlimSAS, MCIO, or retimer BOM.\nDo NOT invent PE pin numbers or assign GCD1 onto S1-S7.\n\nArchitectural names (hierarchical labels; not a fake BGA pinout):\n- PE_S{n}_GCD0_x16 = Conn0 16-lane PCIE bus (OCP-named pads OAM{n}_PCIE_*).\n- PE_S{n}_GCD1_x16 = named only. Overlay Unknown. SERDES_7 as GCD1 PE is Inferred.\n  Pins not assigned. Not S1-S7.\n- PE_SW{k}_US_x16 = four host-facing x16 keepouts toward X11DPH-T.\n\nLane math (verified; not a locked root cause / not a ball map):\n- Full width = 8 modules x 2 GCD x x16 = 256 downstream lanes on the carrier.\n- PM8536B-FEI = 96-lane Gen3, 1311-ball 37.5 mm FCBGA 1.0 mm. Ball map not public.\n- 2x96 = 192. Even with 16 US/switch: 160 DS — enough for 8x x8/GCD (128 DS), NOT 256 DS.\n- 4x96 = 384. Hypothesis partition: each SW 16 US + 64 DS (2 seats x 2 GCD x x16)\n  = 80 of 96, 16 spare. 4 x 16 US = 64 host-facing vs X11DPH-T ~80.\n- Chassis can SIT and be WIRED for 8 full-width. This host CANNOT LIGHT 256 DS.\n  Memory/CPU mix (2x Gold 6230, 64 GB DRAM + 1 TB PMem) does NOT add PCIe lanes.\n- x8/GCD remains a stuffing option if only SW0+SW1 are populated.\n\nSW0 = seats 0-1 (first stuff). SW1 = 2-3. SW2 = 4-5. SW3 = 6-7.\nPEX8780-AB80BI G (80-lane 35 mm) is a cheaper alt in docs only — not placed.\nPM8533B-F3EI (48-lane 27 mm) is a 2-seat alt in docs only — not placed.\n\nX11DPH-T is NOT a part on this PCB. Do not swap or design a host board.\nChamber A B550M is NOT this PCB.\n"
+	(text "PURPOSE: Named v1.0 PCIE_TXnP/N and PCIE_RXnP/N (n=0..15) on ALL 8 seats.\n\nFIRST ARTICLE TARGET: seats 0 and 1. Same 8-seat PCB; 2→4→8 later.\n\nPinmap (Verified OCP v1.0 generic map + pin list; NOT an AMD overlay):\n- Conn0 PCIE_TX/RX0-15 P/N = 64 pads = PETp/n + PERp/n [15:0] \"PCIe or equivalent host link\".\n  That is the only legal named host PE today. Call it GCD0 x16 (architectural name).\n- Conn1 has ZERO PCIE_* pads. S7_* = SERDES_7 \"Reserved Link\" — 64 pads, NO NET.\n  GCD1 x16 is named-only. Do NOT assign S1-S7 as GCD1 PE.\n\nWithout overlay, \"2x MI250X\" on this zip:\n- CAN: two modules SIT on seats 0-1 (mech + named P48V/P12V1/P3V3/GND/GCD0 PE).\n- CAN target at most GCD0 on each (2 GCDs) toward the host keepout.\n- CANNOT: 2 modules at full width (4 GCDs). GCD1 pins Unknown.\n- CANNOT: light even those 2 GCD0 links until Molex 1.2 A/contact is written AND\n  a legal host connector exists. This article does not invent CEM/MCIO.\n\nHost X11DPH-T (NOT on this PCB): 3x Gen3 x16 + 4x Gen3 x8.\n- Two GCD0 x16 (PE_S0_GCD0_x16 + PE_S1_GCD0_x16) FIT the host lane budget.\n- Two full-width modules (4x x16) do NOT.\n\nThis sheet does NOT map pairs onto a CEM x16 pinout.\nDo NOT invent a CEM cable, SlimSAS, MCIO, or retimer BOM.\nDo NOT invent PE pin numbers.\n\nLater seats keep 8-seat names (PE_S2..S7 GCD0/GCD1 + PE_SWk_US_x16) and SW0-SW3 DNP.\n2-module first article does not require stuffing SW0.\n\nX11DPH-T is NOT a part on this PCB. Do not swap or design a host board.\n"
 		(exclude_from_sim no)
 		(at 20.32 20.32 0)
@@
 		(effects (font (size 1.27 1.27)) (justify left))
 	)
+	(hierarchical_label "PE_S1_GCD0_x16"
+		(shape bidirectional)
+		(at 200 138.0 0)
+		(effects (font (size 1.27 1.27)) (justify left))
+	)
+	(hierarchical_label "PE_S0_GCD0_x16"
+		(shape bidirectional)
+		(at 270 130 0)
+		(effects (font (size 1.27 1.27)) (justify left))
+	)
 	(hierarchical_label "PE_S0_GCD1_x16"
 		(shape bidirectional)
-		(at 200 136.0 0)
+		(at 270 136.0 0)
 		(effects (font (size 1.27 1.27)) (justify left))
 	)
 	(hierarchical_label "PE_S1_GCD0_x16"
 		(shape bidirectional)
-		(at 200 142.0 0)
+		(at 270 142.0 0)
 		(effects (font (size 1.27 1.27)) (justify left))
 	)
 	(hierarchical_label "PE_S1_GCD1_x16"
 		(shape bidirectional)
-		(at 200 148.0 0)
+		(at 270 148.0 0)
 		(effects (font (size 1.27 1.27)) (justify left))
 	)
 	(hierarchical_label "PE_S2_GCD0_x16"
 		(shape bidirectional)
-		(at 200 154.0 0)
+		(at 270 154.0 0)
 		(effects (font (size 1.27 1.27)) (justify left))
 	)
 	(hierarchical_label "PE_S2_GCD1_x16"
 		(shape bidirectional)
-		(at 200 160.0 0)
+		(at 270 160.0 0)
 		(effects (font (size 1.27 1.27)) (justify left))
 	)
 	(hierarchical_label "PE_S3_GCD0_x16"
 		(shape bidirectional)
-		(at 200 166.0 0)
+		(at 270 166.0 0)
 		(effects (font (size 1.27 1.27)) (justify left))
 	)
 	(hierarchical_label "PE_S3_GCD1_x16"
 		(shape bidirectional)
-		(at 200 172.0 0)
+		(at 270 172.0 0)
 		(effects (font (size 1.27 1.27)) (justify left))
 	)
 	(hierarchical_label "PE_S4_GCD0_x16"
 		(shape bidirectional)
-		(at 200 178.0 0)
+		(at 270 178.0 0)
 		(effects (font (size 1.27 1.27)) (justify left))
 	)
 	(hierarchical_label "PE_S4_GCD1_x16"
 		(shape bidirectional)
-		(at 200 184.0 0)
+		(at 270 184.0 0)
 		(effects (font (size 1.27 1.27)) (justify left))
 	)
 	(hierarchical_label "PE_S5_GCD0_x16"
 		(shape bidirectional)
-		(at 200 190.0 0)
+		(at 270 190.0 0)
 		(effects (font (size 1.27 1.27)) (justify left))
 	)
 	(hierarchical_label "PE_S5_GCD1_x16"
 		(shape bidirectional)
-		(at 200 196.0 0)
+		(at 270 196.0 0)
 		(effects (font (size 1.27 1.27)) (justify left))
 	)
 	(hierarchical_label "PE_S6_GCD0_x16"
 		(shape bidirectional)
-		(at 200 202.0 0)
+		(at 270 202.0 0)
 		(effects (font (size 1.27 1.27)) (justify left))
 	)
 	(hierarchical_label "PE_S6_GCD1_x16"
 		(shape bidirectional)
-		(at 200 208.0 0)
+		(at 270 208.0 0)
 		(effects (font (size 1.27 1.27)) (justify left))
 	)
 	(hierarchical_label "PE_S7_GCD0_x16"
 		(shape bidirectional)
-		(at 200 214.0 0)
+		(at 270 214.0 0)
 		(effects (font (size 1.27 1.27)) (justify left))
 	)
 	(hierarchical_label "PE_S7_GCD1_x16"
 		(shape bidirectional)
-		(at 200 220.0 0)
+		(at 270 220.0 0)
 		(effects (font (size 1.27 1.27)) (justify left))
 	)
 	(hierarchical_label "PE_SW0_US_x16"
 		(shape bidirectional)
-		(at 200 226.0 0)
+		(at 270 226.0 0)
 		(effects (font (size 1.27 1.27)) (justify left))
 	)
 	(hierarchical_label "PE_SW1_US_x16"
 		(shape bidirectional)
-		(at 200 232.0 0)
+		(at 270 232.0 0)
 		(effects (font (size 1.27 1.27)) (justify left))
 	)
 	(hierarchical_label "PE_SW2_US_x16"
 		(shape bidirectional)
-		(at 200 238.0 0)
+		(at 270 238.0 0)
 		(effects (font (size 1.27 1.27)) (justify left))
 	)
 	(hierarchical_label "PE_SW3_US_x16"
 		(shape bidirectional)
-		(at 200 244.0 0)
-		(effects (font (size 1.27 1.27)) (justify left))
-	)
+		(at 270 244.0 0)
+		(effects (font (size 1.27 1.27)) (justify left))
+	)
